File: PCBs/Transmitter Rev 1.sch (EAGLE design)
At the start: 20 parts, among them J1 U.FL-R-SMT(01), U1 RFM95W-868S2, U2 TSRN_1-2450

Commit message: Finalize schematic
Parts:
- removed ANT1: CHIP_ANTENNA, RTR:CHIP_ANTENNA
- removed J1: U.FL-R-SMT(01), RTR:U.FL-R-SMT(01)
- added 5V_BOOST_CONVERTER: TPS61032PWPR, RTR:TPS61032PWPR
- added ALT_SWITCH, ALT_SWITCH1: JP-2C, RTR:JP-2C
- added BATTERY_PROTECTION: BQ29700DSER, RTR:BQ29700DSER
- added CHARGE_CONTROLLER: MCP73831T-2ACI/MC, RTR:MCP73831T-2ACI/MC
- added CHG_C1, CHG_C2: 4.7uF, RTR:C-SMD
- added CHG_C3: .1uF, RTR:C-SMD
- added CHG_C4: 10uF, RTR:C-SMD
- added CHG_C5: 2.2uF, RTR:C-SMD
- added CHG_C6: 220uF, RTR:C-SMD
- added CHG_R1: 2k, RTR:R-SMD
- added CHG_R2, CHG_R5: 470, RTR:R-SMD
- added CHG_R3: 330, RTR:R-SMD
- added CHG_R4: 2.2k, RTR:R-SMD
- added CHG_STAT, PWR_STAT: (no value), RTR:LED5MM
- added CHIP_ANTENNA: ANT1204LL05R0915A, RTR:ANT1204LL05R0915A
- added L2: 6.8uH, RTR:L_SMD
- added SW1, SW2: SCREW_SWITCH, RTR:SCREW_SWITCH
- added U5: DMG9926USD-13, RTR:DMG9926USD-13
- added UFL_CON: U.FL-R-SMT(01), RTR:U.FL-R-SMT(01)
- 9V_CON, ANT_CON: value (none) -> JP-2C; device RTR:JP2E -> RTR:JP-2C
- ANALOG, I2C1, I2C2, SPI1.2, UART1, UART2: device RTR:SENSOR_CONNECTORPTH_FEMALE -> RTR:SENSOR_BREAKOUTPTH_FEMALE
- L1: device RTR:L -> RTR:L_SMD
- SPI1: value 2X6 FEMALE -> SNSR_BRKOUT; device RTR:SENSOR_CONNECTORPTH_FEMALE -> RTR:SENSOR_BREAKOUTPTH_FEMALE
Connections:
- new net LI-PO_5V_OUT: 5V_BOOST_CONVERTER.VOUT, 9V_CON.1, ALT_SWITCH.2, CHG_C5.1, CHG_C6.1, SW1.2
- new net N$10: CHG_R2.2, CHG_STAT.C
- new net N$11: CHARGE_CONTROLLER.PROG, CHG_R1.1
- new net N$12: BATTERY_PROTECTION.BAT, CHG_C3.1, CHG_R3.2
- new net N$13: 5V_BOOST_CONVERTER.EN, 5V_BOOST_CONVERTER.SYNC, 5V_BOOST_CONVERTER.VBAT, CHARGE_CONTROLLER.VBAT, CHG_C2.1, CHG_C4.1, CHG_R3.1, L2.1, LIPO.+
- new net N$14: BATTERY_PROTECTION.VSS, CHG_C3.2, LIPO.-, U5.S2
- new net N$15: U5.D1, U5.D2
- new net N$16: BATTERY_PROTECTION.DOUT, U5.G2
- new net N$17: BATTERY_PROTECTION.V-, CHG_R4.2
- new net N$18: BATTERY_PROTECTION.COUT, U5.G1
- new net N$19: ALT_SWITCH.3, BRD1.USB1_VI, PWR_STAT.A, SW1.1
- new net N$20: 5V_BOOST_CONVERTER.SW, L2.2
- new net N$22: ALT_SWITCH1.3, BRD1.BAT_VIN, SW2.1
- new net N$9: CHARGE_CONTROLLER.STAT, CHG_R2.1
- net GND: now also 5V_BOOST_CONVERTER.GND, 5V_BOOST_CONVERTER.LBI, 5V_BOOST_CONVERTER.PGND, 5V_BOOST_CONVERTER.PWRPAD, CHARGE_CONTROLLER.VSS, CHG_C1.2, CHG_C2.2, CHG_C4.2, CHG_C5.2, CHG_C6.2, CHG_R1.2, CHG_R4.1, CHG_R5.1, U5.S1
- net N$2: now also CHIP_ANTENNA.ANT; no longer ANT1.ANT
- net N$3: now also UFL_CON.GND, UFL_CON.SIG; no longer J1.GND, J1.SIG
- net N$4: now also ALT_SWITCH1.2, SW2.2; no longer BRD1.BAT_VIN
- net N$8: now also CHG_R5.2, PWR_STAT.C; no longer 9V_CON.1, BRD1.VIN
- net VCC_5V: now also CHARGE_CONTROLLER.VDD, CHG_C1.1, CHG_STAT.A
Other:
- note added: "9V POWER"
- note added: "EXPANSION PORTS"
- note added: "IMPORTANT: Turn off Switch BEFORE plugging in USB! Not following this could severely damage the board!"
- note added: "LI-PO POWER"
- note added: "POCKET-BEAGLE"
- note added: "RF"
- note added: "RICE ECLIPSE REAL TIME ROCKET TRANSMITTER REV 1"
- moved on the sheet: ALT_9V, ALT_PWR, ANALOG, ANT_CON, I2C1, I2C2, LIPO, SPI1, SPI1.2, U1, U2, UART1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

Commit message: Update datasheets, small schematic revisions, add test pins
Parts:
- added T1, T2, T3, T4, T5, T6, T7: TEST_PAD, RTR:TEST_PAD
Connections:
- net GND: now also T2.P$1, UFL_CON.GND
- net LI-PO_5V_OUT: now also T6.P$1
- net N$13: now also T4.P$1
- net N$14: now also T5.P$1
- net N$19: now also T7.P$1
- net N$3: no longer UFL_CON.GND
- net VCC: now also T1.P$1
- net VCC_5V: now also T3.P$1
Changed lines of the file:
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@@
 <part name="PWR_STAT" library="RTR" deviceset="LED" device="5MM" package3d_urn="urn:adsk.eagle:package:15799/2"/>
 <part name="CHG_R5" library="RTR" deviceset="R-SMD" device="" value="470"/>
+<part name="GND17" library="RTR" deviceset="GND" device=""/>
+<part name="P+11" library="RTR" deviceset="VCC" device=""/>
+<part name="T1" library="RTR" deviceset="TEST_PAD" device=""/>
+<part name="T2" library="RTR" deviceset="TEST_PAD" device=""/>
+<part name="T3" library="RTR" deviceset="TEST_PAD" device=""/>
+<part name="T4" library="RTR" deviceset="TEST_PAD" device=""/>
+<part name="T5" library="RTR" deviceset="TEST_PAD" device=""/>
+<part name="T6" library="RTR" deviceset="TEST_PAD" device=""/>
+<part name="T7" library="RTR" deviceset="TEST_PAD" device=""/>
 </parts>
 <sheets>
@@
 <attribute name="VALUE" x="21.082" y="3.81" size="1.778" layer="96" rot="R90"/>
 </instance>
+<instance part="GND17" gate="1" x="228.6" y="-22.86" smashed="yes"/>
+<instance part="P+11" gate="VCC" x="213.36" y="-7.62" smashed="yes"/>
+<instance part="T1" gate="G$1" x="220.98" y="-12.7" smashed="yes">
+<attribute name="NAME" x="215.9" y="-7.62" size="1.778" layer="95"/>
+</instance>
+<instance part="T2" gate="G$1" x="228.6" y="-12.7" smashed="yes">
+<attribute name="NAME" x="223.52" y="-7.62" size="1.778" layer="95"/>
+</instance>
+<instance part="T3" gate="G$1" x="-127" y="-106.68" smashed="yes">
+<attribute name="NAME" x="-132.08" y="-101.6" size="1.778" layer="95"/>
+</instance>
+<instance part="T4" gate="G$1" x="0" y="-101.6" smashed="yes">
+<attribute name="NAME" x="-5.08" y="-96.52" size="1.778" layer="95"/>
+</instance>
+<instance part="T5" gate="G$1" x="20.32" y="-137.16" smashed="yes">
+<attribute name="NAME" x="15.24" y="-132.08" size="1.778" layer="95"/>
+</instance>
+<instance part="T6" gate="G$1" x="180.34" y="-101.6" smashed="yes">
+<attribute name="NAME" x="175.26" y="-96.52" size="1.778" layer="95"/>
+</instance>
+<instance part="T7" gate="G$1" x="33.02" y="45.72" smashed="yes">
+<attribute name="NAME" x="27.94" y="48.26" size="1.778" layer="95"/>
+</instance>
 </instances>
 <busses>
@@
 <junction x="-106.68" y="-109.22"/>
 <label x="-121.92" y="-109.22" size="1.778" layer="95"/>
+<pinref part="T3" gate="G$1" pin="P$1"/>
 </segment>
 </net>
@@
 <wire x1="-71.12" y1="-48.26" x2="-76.2" y2="-48.26" width="0.1524" layer="91"/>
 <wire x1="-76.2" y1="-48.26" x2="-76.2" y2="-45.72" width="0.1524" layer="91"/>
+</segment>
+<segment>
+<pinref part="P+11" gate="VCC" pin="VCC"/>
+<wire x1="213.36" y1="-10.16" x2="213.36" y2="-15.24" width="0.1524" layer="91"/>
+<wire x1="213.36" y1="-15.24" x2="220.98" y2="-15.24" width="0.1524" layer="91"/>
+<pinref part="T1" gate="G$1" pin="P$1"/>
 </segment>
 </net>
@@
 <wire x1="-48.26" y1="93.98" x2="-45.72" y2="93.98" width="0.1524" layer="91"/>
 <junction x="-45.72" y="93.98"/>
+<pinref part="UFL_CON" gate="G$1" pin="GND"/>
+<wire x1="-15.24" y1="104.14" x2="-15.24" y2="96.52" width="0.1524" layer="91"/>
+<wire x1="-15.24" y1="96.52" x2="-45.72" y2="96.52" width="0.1524" layer="91"/>
+<junction x="-45.72" y="96.52"/>
 </segment>
 <segment>
@@
 <junction x="101.6" y="-137.16"/>
 </segment>
+<segment>
+<pinref part="GND17" gate="1" pin="GND"/>
+<wire x1="228.6" y1="-15.24" x2="228.6" y2="-20.32" width="0.1524" layer="91"/>
+<pinref part="T2" gate="G$1" pin="P$1"/>
+</segment>
 </net>
 <net name="RF_RST" class="0">
@@
 <net name="N$3" class="0">
 <segment>
+<pinref part="ANT_CON" gate="1" pin="1"/>
+<wire x1="-30.48" y1="109.22" x2="-15.24" y2="109.22" width="0.1524" layer="91"/>
 <pinref part="UFL_CON" gate="G$1" pin="SIG"/>
-<pinref part="UFL_CON" gate="G$1" pin="GND"/>
-<wire x1="-15.24" y1="104.14" x2="-15.24" y2="106.68" width="0.1524" layer="91"/>
-<pinref part="ANT_CON" gate="1" pin="1"/>
-<wire x1="-15.24" y1="106.68" x2="-15.24" y2="109.22" width="0.1524" layer="91"/>
-<wire x1="-30.48" y1="109.22" x2="-17.78" y2="109.22" width="0.1524" layer="91"/>
-<wire x1="-17.78" y1="109.22" x2="-17.78" y2="106.68" width="0.1524" layer="91"/>
-<wire x1="-17.78" y1="106.68" x2="-15.24" y2="106.68" width="0.1524" layer="91"/>
-<junction x="-15.24" y="106.68"/>
 </segment>
 </net>
@@
 <junction x="-25.4" y="-109.22"/>
 <wire x1="-25.4" y1="-109.22" x2="-25.4" y2="-104.14" width="0.1524" layer="91"/>
-<wire x1="-25.4" y1="-104.14" x2="78.74" y2="-104.14" width="0.1524" layer="91"/>
 <pinref part="5V_BOOST_CONVERTER" gate="G$1" pin="SYNC"/>
+<wire x1="-25.4" y1="-104.14" x2="0" y2="-104.14" width="0.1524" layer="91"/>
+<wire x1="0" y1="-104.14" x2="78.74" y2="-104.14" width="0.1524" layer="91"/>
 <wire x1="106.68" y1="-119.38" x2="99.06" y2="-119.38" width="0.1524" layer="91"/>
 <pinref part="5V_BOOST_CONVERTER" gate="G$1" pin="VBAT"/>
@@
 <junction x="99.06" y="-109.22"/>
 <junction x="78.74" y="-109.22"/>
+<pinref part="T4" gate="G$1" pin="P$1"/>
+<junction x="0" y="-104.14"/>
 </segment>
 </net>
@@
 <segment>
 <pinref part="LIPO" gate="G$1" pin="-"/>
+<pinref part="U5" gate="G$1" pin="S2"/>
+<wire x1="48.26" y1="-139.7" x2="20.32" y2="-139.7" width="0.1524" layer="91"/>
+<wire x1="20.32" y1="-139.7" x2="0" y2="-139.7" width="0.1524" layer="91"/>
+<wire x1="0" y1="-139.7" x2="-25.4" y2="-139.7" width="0.1524" layer="91"/>
+<wire x1="-25.4" y1="-139.7" x2="-25.4" y2="-124.46" width="0.1524" layer="91"/>
 <pinref part="BATTERY_PROTECTION" gate="G$1" pin="VSS"/>
-<wire x1="-25.4" y1="-119.38" x2="-10.16" y2="-119.38" width="0.1524" layer="91"/>
+<wire x1="-25.4" y1="-124.46" x2="-25.4" y2="-119.38" width="0.1524" layer="91"/>
+<wire x1="0" y1="-119.38" x2="0" y2="-139.7" width="0.1524" layer="91"/>
+<junction x="0" y="-139.7"/>
 <pinref part="CHG_C3" gate="G$1" pin="2"/>
-<wire x1="-10.16" y1="-119.38" x2="0" y2="-119.38" width="0.1524" layer="91"/>
-<junction x="-10.16" y="-119.38"/>
-<junction x="-25.4" y="-119.38"/>
-<pinref part="U5" gate="G$1" pin="S2"/>
-<wire x1="48.26" y1="-139.7" x2="-25.4" y2="-139.7" width="0.1524" layer="91"/>
-<wire x1="-25.4" y1="-139.7" x2="-25.4" y2="-119.38" width="0.1524" layer="91"/>
+<wire x1="-10.16" y1="-119.38" x2="-10.16" y2="-124.46" width="0.1524" layer="91"/>
+<wire x1="-10.16" y1="-124.46" x2="-25.4" y2="-124.46" width="0.1524" layer="91"/>
+<junction x="-25.4" y="-124.46"/>
+<pinref part="T5" gate="G$1" pin="P$1"/>
+<junction x="20.32" y="-139.7"/>
 </segment>
 </net>
@@
 <wire x1="157.48" y1="-109.22" x2="157.48" y2="-104.14" width="0.1524" layer="91"/>
 <junction x="157.48" y="-104.14"/>
-<wire x1="172.72" y1="-104.14" x2="198.12" y2="-104.14" width="0.1524" layer="91"/>
 <junction x="172.72" y="-104.14"/>
 <label x="182.88" y="-104.14" size="1.778" layer="95"/>
+<wire x1="172.72" y1="-104.14" x2="180.34" y2="-104.14" width="0.1524" layer="91"/>
+<pinref part="T6" gate="G$1" pin="P$1"/>
+<wire x1="180.34" y1="-104.14" x2="198.12" y2="-104.14" width="0.1524" layer="91"/>
+<junction x="180.34" y="-104.14"/>
 </segment>
 <segment>
@@
 <wire x1="20.32" y1="43.18" x2="22.86" y2="43.18" width="0.1524" layer="91"/>
 <pinref part="PWR_STAT" gate="G$1" pin="A"/>
-<wire x1="22.86" y1="43.18" x2="55.88" y2="43.18" width="0.1524" layer="91"/>
+<wire x1="22.86" y1="43.18" x2="33.02" y2="43.18" width="0.1524" layer="91"/>
+<wire x1="33.02" y1="43.18" x2="55.88" y2="43.18" width="0.1524" layer="91"/>
 <wire x1="22.86" y1="20.32" x2="22.86" y2="43.18" width="0.1524" layer="91"/>
 <junction x="22.86" y="43.18"/>
-</segment>
-</net>
+<pinref part="T7" gate="G$1" pin="P$1"/>
+<junction x="33.02" y="43.18"/>
+</segment>
+</net>

Commit message: Lay out components logically on board, miscellaneous library and schematic additions and fixes
Parts:
- removed CHG_R3: 330, RTR:R-SMD
- removed CHG_R4: 2.2k, RTR:R-SMD
- removed CHG_R5: 470, RTR:R-SMD
- removed L1: 5.6uH, RTR:L_SMD
- removed SW1, SW2: SCREW_SWITCH, RTR:SCREW_SWITCH
- added 9V_L1: 5.6uH, RTR:L_SMD
- added ANALOG_BRK, I2C1_BRK, I2C2_BRK, SPI1.2_BRK, SPI1_BRK, UART1_BRK, UART2_BRK: SENSOR_PIN_BREAKOUT, RTR:SENSOR_PIN_BREAKOUT
- added BAT_PWR: SCREW_SWITCH, RTR:SCREW_SWITCH
- added BAT_R1: 330, RTR:R-SMD1206
- added BAT_R2: 2.2k, RTR:R-SMD1206
- added J1: 10118193-0001LF, RTR:10118193-0001LF
- added LED_R_1: 470, RTR:R-SMD1206
- added PWR_C1: 10uF, RTR:C-SMD
- added RF_C1: .1uF, RTR:C-SMD
- added T10, T8, T9: TEST_PAD, RTR:TEST_PAD
- CHG_R1: value 2k -> 470; device RTR:R-SMD -> RTR:R-SMD1206
- CHG_R2: value 470 -> 2k; device RTR:R-SMD -> RTR:R-SMD1206
- SPI1: value SNSR_BRKOUT -> 2X6 FEMALE
- renumbered CHG_C3 to BAT_C1, CHG_C4 to CONV_C1, CHG_C5 to CONV_C2, CHG_C6 to CONV_C3, L2 to CONV_L1, U5 to DUAL_N_MOSFETS
Connections:
- net N$1 renamed RF_ANT
- net N$14 renamed LI-PO_-
- net N$16 renamed DOUT
- net N$18 renamed COUT
- net N$2 renamed ANT
- removed net N$10: CHG_R2.2, CHG_STAT.C
- removed net N$11: CHARGE_CONTROLLER.PROG, CHG_R1.1
- removed net N$12: BATTERY_PROTECTION.BAT, BAT_C1.1, CHG_R3.2
- removed net N$13: 5V_BOOST_CONVERTER.EN, 5V_BOOST_CONVERTER.SYNC, 5V_BOOST_CONVERTER.VBAT, CHARGE_CONTROLLER.VBAT, CHG_C2.1, CHG_R3.1, CONV_C1.1, CONV_L1.1, LIPO.+, T4.P$1
- removed net N$15: DUAL_N_MOSFETS.D1, DUAL_N_MOSFETS.D2
- removed net N$17: BATTERY_PROTECTION.V-, CHG_R4.2
- removed net N$19: ALT_SWITCH.3, BRD1.USB1_VI, PWR_STAT.A, SW1.1, T7.P$1
- removed net N$22: ALT_SWITCH1.3, BRD1.BAT_VIN, SW2.1
- removed net N$3: ANT_CON.1, UFL_CON.SIG
- removed net N$4: 9V_CON.3, ALT_PWR.+, ALT_SWITCH1.2, SW2.2
- removed net N$5: 9V_CON.2, U2.VOUT
- removed net N$6: 9V_C2.1, L1.2, U2.VIN
- removed net N$7: 9V_C1.1, ALT_9V.+, L1.1
- removed net N$8: CHG_R5.2, PWR_STAT.C
- removed net N$9: CHARGE_CONTROLLER.STAT, CHG_R2.1
- new net 9V_+: 9V_C1.1, 9V_L1.1, ALT_9V.+
- new net 9V_VIN: 9V_C2.1, 9V_L1.2, U2.VIN
- new net 9V_VOUT: 9V_CON.2, T9.P$1, U2.VOUT
- new net ALT_PWR_+: 9V_CON.3, ALT_PWR.+, ALT_SWITCH1.2
- new net BAT: BATTERY_PROTECTION.BAT, BAT_C1.1, BAT_R1.2
- new net BAT_VIN: ALT_SWITCH1.3, BRD1.BAT_VIN
- new net LED: LED_R_1.2, PWR_STAT.C
- new net LED-: CHG_R1.2, CHG_STAT.C
- new net LI-PO_+: 5V_BOOST_CONVERTER.EN, 5V_BOOST_CONVERTER.SYNC, 5V_BOOST_CONVERTER.VBAT, BAT_R1.1, CHARGE_CONTROLLER.VBAT, CHG_C2.1, CONV_C1.1, CONV_L1.1, LIPO.+, T4.P$1
- new net N$21: SPI1.14, SPI1_BRK.2
- new net N$23: SPI1.13, SPI1_BRK.1
- new net N$24: SPI1.15, SPI1_BRK.3
- new net N$25: SPI1.16, SPI1_BRK.4
- new net N$26: SPI1.2.13, SPI1.2_BRK.1
- new net N$27: SPI1.2.14, SPI1.2_BRK.2
- new net N$28: SPI1.2.16, SPI1.2_BRK.4
- new net N$29: SPI1.2.15, SPI1.2_BRK.3
- new net N$30: UART1.13, UART1_BRK.1
- new net N$31: UART1.15, UART1_BRK.3
- new net N$32: UART1.14, UART1_BRK.2
- new net N$33: UART1.16, UART1_BRK.4
- new net N$35: UART2.15, UART2_BRK.3
- new net N$36: UART2.16, UART2_BRK.4
- new net N$37: UART2.14, UART2_BRK.2
- new net N$38: UART2.13, UART2_BRK.1
- new net N$39: I2C1.16, I2C1_BRK.4
- new net N$40: I2C1.15, I2C1_BRK.3
- new net N$41: I2C1.13, I2C1_BRK.1
- new net N$42: I2C1.14, I2C1_BRK.2
- new net N$43: I2C2.15, I2C2_BRK.3
- new net N$44: I2C2.16, I2C2_BRK.4
- new net N$45: I2C2.14, I2C2_BRK.2
- new net N$46: I2C2.13, I2C2_BRK.1
- new net N$47: ANALOG.15, ANALOG_BRK.3
- new net N$48: ANALOG.16, ANALOG_BRK.4
- new net N$49: ANALOG.14, ANALOG_BRK.2
- new net N$50: ANALOG.13, ANALOG_BRK.1
- new net PROG: CHARGE_CONTROLLER.PROG, CHG_R2.1
- new net SOURCE: DUAL_N_MOSFETS.D1, DUAL_N_MOSFETS.D2, T10.P$1
- new net STAT: CHARGE_CONTROLLER.STAT, CHG_R1.1
- new net SWITCH_5V: ALT_SWITCH.3, BAT_PWR.1, BRD1.USB1_VI, PWR_C1.1, PWR_STAT.A, T7.P$1
- new net UFL: ANT_CON.1, T8.P$1, UFL_CON.SIG
- new net V-: BATTERY_PROTECTION.V-, BAT_R2.2
- new net V_USB: CHARGE_CONTROLLER.VDD, CHG_C1.1, CHG_STAT.A, J1.VUSB, T3.P$1
- net GND: now also BAT_R2.1, CHARGE_CONTROLLER.EP, CHG_R2.2, J1.GND, LED_R_1.1, PWR_C1.2, RF_C1.2; no longer CHG_R1.2, CHG_R4.1, CHG_R5.1
- net LI-PO_5V_OUT: now also BAT_PWR.2; no longer SW1.2
- net VCC: now also RF_C1.1
- net VCC_5V: no longer CHARGE_CONTROLLER.VDD, CHG_C1.1, CHG_STAT.A, T3.P$1
Other:
- moved on the sheet: ALT_9V, ANT_CON, CHIP_ANTENNA, T3, U1, U2, UFL_CON

Commit message: Route Board
Connections:
- net SOURCE renamed DRAIN
- net UFL renamed N$1
Other:
- moved on the sheet: T10, T3, T4, T5, T6, T7, T8, T9
