File: PCBs/Electro Transmitter Rev 1.brd (EAGLE design)
At the start: 113 x 63.5 mm, 62 parts, among them J1 10118193-0001LF, T1 TEST_PAD, T10 TEST_PAD, T2 TEST_PAD, T3 TEST_PAD, T4 TEST_PAD, T5 TEST_PAD, T6 TEST_PAD, T7 TEST_PAD, T8 TEST_PAD, T9 TEST_PAD, U1 RFM95W-868S2, U2 TSRN_1-2450

Commit message: GPS2 schematic
Parts:
- SPI1: device RTR:2X7 -> RTR Main Library:2X7
Changed lines of the file:
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@@
 <attribute name="VALUE" x="5.7658" y="54.9148" size="1.27" layer="27" ratio="10" rot="R180"/>
 </element>
-<element name="SPI1" library="RTR" package="2X7" package3d_urn="urn:adsk.eagle:package:38277/1" value="2X6 FEMALE" x="24.13" y="50.8" smashed="yes">
+<element name="SPI1" library="RTR Main Library" package="2X7" package3d_urn="urn:adsk.eagle:package:38277/1" value="2X6 FEMALE" x="24.13" y="50.8" smashed="yes">
 <attribute name="NAME" x="22.606" y="62.103" size="1.27" layer="25" font="vector" ratio="20"/>
 <attribute name="PROD_ID" value="CONN-12423" x="102.87" y="-21.59" size="1.778" layer="27" display="off"/>
@@
 <wire x1="74.549" y1="38.9001" x2="74.549" y2="38.735" width="1.016" layer="1"/>
 <wire x1="80.57515" y1="44.92625" x2="74.549" y2="38.9001" width="1.016" layer="1"/>
+<wire x1="72.898" y1="38.989" x2="74.549" y2="38.735" width="0" layer="19" extent="16-16"/>
+<wire x1="2.032" y1="27.94" x2="6.226" y2="26.162" width="0" layer="19" extent="1-1"/>
+<wire x1="2.483" y1="33.925" x2="2.708" y2="32.06" width="0" layer="19" extent="1-1"/>
+<wire x1="2.483" y1="34.925" x2="2.483" y2="33.925" width="0" layer="19" extent="1-1"/>
+<wire x1="2.483" y1="35.925" x2="2.483" y2="34.925" width="0" layer="19" extent="1-1"/>
+<wire x1="3.683" y1="35.925" x2="2.483" y2="35.925" width="0" layer="19" extent="1-1"/>
+<wire x1="3.683" y1="34.925" x2="3.683" y2="35.925" width="0" layer="19" extent="1-1"/>
+<wire x1="3.683" y1="33.925" x2="3.683" y2="34.925" width="0" layer="19" extent="1-1"/>
+<wire x1="4.883" y1="35.925" x2="3.683" y2="35.925" width="0" layer="19" extent="1-1"/>
+<wire x1="4.883" y1="34.925" x2="4.883" y2="35.925" width="0" layer="19" extent="1-1"/>
+<wire x1="4.883" y1="33.925" x2="4.883" y2="34.925" width="0" layer="19" extent="1-1"/>
+<wire x1="8.865" y1="41.656" x2="7.112" y2="40.767" width="0" layer="19" extent="16-16"/>
+<wire x1="8.509" y1="48.26" x2="9.779" y2="48.895" width="0" layer="19" extent="16-16"/>
+<wire x1="8.255" y1="49.022" x2="8.509" y2="48.26" width="0" layer="19" extent="16-16"/>
+<wire x1="16.637" y1="47.436" x2="9.779" y2="48.895" width="0" layer="19" extent="16-16"/>
+<wire x1="18.186" y1="46.99" x2="16.637" y2="47.436" width="0" layer="19" extent="1-16"/>
+<wire x1="20.196" y1="37.211" x2="18.926" y2="39.37" width="0" layer="19" extent="1-1"/>
+<wire x1="76.835" y1="29.845" x2="74.549" y2="38.735" width="0" layer="19" extent="1-1"/>
+<wire x1="27.94" y1="55.88" x2="20.193" y2="47.117" width="0" layer="19" extent="1-1"/>
+<wire x1="53.34" y1="55.88" x2="52.705" y2="53.34" width="0" layer="19" extent="16-16"/>
+<wire x1="81.2714" y1="15.8092" x2="81.2714" y2="29.8092" width="0" layer="19" extent="1-1"/>
+<wire x1="86.233" y1="11.938" x2="80.515" y2="12.827" width="0" layer="19" extent="1-1"/>
+<wire x1="45.466" y1="20.574" x2="45.466" y2="18.034" width="0" layer="19" extent="1-1"/>
+<wire x1="53.086" y1="20.574" x2="45.466" y2="20.574" width="0" layer="19" extent="1-1"/>
 </signal>
 <signal name="RF_RST">
