File: PCBs/Electro Transmitter Rev 1.sch (EAGLE design)
At the start: 61 parts, among them J1 10118193-0001LF, T1 TEST_PAD, T10 TEST_PAD, T2 TEST_PAD, T3 TEST_PAD, T4 TEST_PAD, T5 TEST_PAD, T6 TEST_PAD, T7 TEST_PAD, T8 TEST_PAD, T9 TEST_PAD, U1 RFM95W-868S2, U2 TSRN_1-2450

Commit message: GPS2 schematic
Parts:
- SPI1: device RTR:SENSOR_BREAKOUTPTH_FEMALE -> RTR Main Library:SENSOR_BREAKOUTPTH_FEMALE
Changed lines of the file:
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@@
 <part name="UFL_CON" library="RTR" deviceset="U.FL-R-SMT(01)" device=""/>
 <part name="P+2" library="RTR" deviceset="VCC" device=""/>
-<part name="SPI1" library="RTR" deviceset="SENSOR_BREAKOUT" device="PTH_FEMALE" package3d_urn="urn:adsk.eagle:package:38277/1" value="2X6 FEMALE"/>
+<part name="SPI1" library="RTR Main Library" deviceset="SENSOR_BREAKOUT" device="PTH_FEMALE" package3d_urn="urn:adsk.eagle:package:38277/1" value="2X6 FEMALE"/>
 <part name="UART1" library="RTR" deviceset="SENSOR_BREAKOUT" device="PTH_FEMALE" package3d_urn="urn:adsk.eagle:package:38277/1" value="2X6 FEMALE"/>
 <part name="UART2" library="RTR" deviceset="SENSOR_BREAKOUT" device="PTH_FEMALE" package3d_urn="urn:adsk.eagle:package:38277/1" value="2X6 FEMALE"/>
