File: PCBs/ElectroII (UPDATE).brd (EAGLE design)
At the start: 114.3 x 76.2 mm, 33 parts, among them IC1 TLF50211ELXUMA2, J1 U.FL-R-SMT(01), T1 VBAT, T2 BUCK, T3 GND, T5 VCC, T7 5V, U1 RFM95W-868S2

Commit message: fixed with erc and drc
should be go to go
Connections:
- removed net BUCK_OUT: C_OUT.1, DOUT.A, L_OUT.P$2, PWR.A, T2.P$1
- net FB: now also C_OUT.1, DOUT.A, L_OUT.P$2, PWR.A, T2.P$1
Routing:
- net FB: track 0.00 -> 39.9 mm
- net BUCK_OUT: track 23.4 -> 0.00 mm
- net 5V: track 211.8 -> 212.7 mm, vias 4 -> 5
Changed lines of the file:
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@@
 <wire x1="54.7878" y1="43.6626" x2="54.725" y2="43.645" width="0.508" layer="1"/>
 <wire x1="57.2262" y1="43.6626" x2="57.265" y2="43.645" width="0.508" layer="1"/>
-<wire x1="32.9946" y1="34.29" x2="32.9946" y2="23.368" width="0.508" layer="16"/>
+<wire x1="32.9946" y1="23.368" x2="32.9946" y2="34.29" width="0.508" layer="16"/>
 <wire x1="32.9946" y1="23.368" x2="32.9946" y2="7.62" width="0.508" layer="16"/>
-<wire x1="31.7754" y1="35.5092" x2="32.9946" y2="34.29" width="0.508" layer="16"/>
 <wire x1="32.9946" y1="7.62" x2="33.02" y2="7.62" width="0.508" layer="16"/>
 <wire x1="55.3212" y1="7.62" x2="59.69" y2="7.62" width="0.508" layer="1"/>
@@
 <wire x1="52.3494" y1="43.6626" x2="54.7116" y2="43.6626" width="0.508" layer="16"/>
 <wire x1="50.9778" y1="45.0342" x2="52.3494" y2="43.6626" width="0.508" layer="16"/>
-<wire x1="42.3672" y1="45.0342" x2="50.9778" y2="45.0342" width="0.508" layer="16"/>
-<wire x1="32.4612" y1="35.1282" x2="42.3672" y2="45.0342" width="0.508" layer="16"/>
+<wire x1="50.9778" y1="45.0342" x2="42.3672" y2="45.0342" width="0.508" layer="16"/>
 <wire x1="54.7116" y1="43.6626" x2="54.725" y2="43.645" width="0.508" layer="16"/>
 <wire x1="30.48" y1="57.6834" x2="30.48" y2="68.58" width="0.508" layer="16"/>
 <wire x1="29.4894" y1="56.6928" x2="30.48" y2="57.6834" width="0.508" layer="16"/>
-<wire x1="29.4894" y1="37.7952" x2="29.4894" y2="56.6928" width="0.508" layer="1"/>
-<wire x1="31.5468" y1="35.7378" x2="29.4894" y2="37.7952" width="0.508" layer="1"/>
+<wire x1="29.4894" y1="56.6928" x2="29.4894" y2="37.7952" width="0.508" layer="1"/>
 <via x="38.7096" y="64.389" extent="1-16" drill="0.35"/>
 <via x="86.2584" y="69.8754" extent="1-16" drill="0.35"/>
@@
 <wire x1="29.9466" y1="20.32" x2="32.9946" y2="23.368" width="0.508" layer="16"/>
 <wire x1="18.796" y1="20.32" x2="13.97" y2="20.32" width="0.508" layer="1"/>
-<wire x1="31.7754" y1="35.5092" x2="32.4612" y2="35.1282" width="0" layer="19" extent="16-16"/>
-<wire x1="31.5468" y1="35.7378" x2="31.7754" y2="35.5092" width="0" layer="19" extent="1-16"/>
+<wire x1="29.4894" y1="37.7952" x2="29.4894" y2="37.0586" width="0.4572" layer="1"/>
+<wire x1="31.4198" y1="35.1282" x2="32.4612" y2="35.1282" width="0.4572" layer="1"/>
+<via x="32.4612" y="35.1282" extent="1-16" drill="0.35"/>
+<wire x1="29.4894" y1="37.0586" x2="31.4198" y2="35.1282" width="0.4572" layer="1"/>
+<wire x1="42.3672" y1="45.0342" x2="32.4612" y2="35.1282" width="0.4572" layer="16"/>
+<wire x1="32.9946" y1="34.29" x2="32.9946" y2="34.5948" width="0.4572" layer="16"/>
+<wire x1="32.9946" y1="34.5948" x2="32.4612" y2="35.1282" width="0.4572" layer="16"/>
 </signal>
 <signal name="TX">
@@
 <signal name="FB">
 <contactref element="IC1" pad="7"/>
+<contactref element="L_OUT" pad="P$2"/>
+<contactref element="C_OUT" pad="1"/>
+<contactref element="T2" pad="P$1"/>
+<contactref element="PWR" pad="A"/>
+<contactref element="DOUT" pad="A"/>
+<wire x1="18.796" y1="30.48" x2="18.796" y2="34.798" width="0.508" layer="1"/>
+<wire x1="18.796" y1="34.798" x2="18.796" y2="36.706" width="0.508" layer="1"/>
+<wire x1="18.796" y1="36.706" x2="18.92" y2="36.83" width="0.508" layer="1"/>
+<wire x1="18.92" y1="36.83" x2="18.92" y2="44.397" width="0.508" layer="1"/>
+<wire x1="18.92" y1="44.397" x2="18.973" y2="44.45" width="0.508" layer="1"/>
+<wire x1="18.973" y1="44.45" x2="22.86" y2="44.45" width="0.508" layer="1"/>
+<wire x1="22.86" y1="44.45" x2="22.987" y2="44.323" width="0.508" layer="1"/>
+<wire x1="18.796" y1="34.798" x2="20.447" y2="34.798" width="0.508" layer="1"/>
+<wire x1="20.447" y1="34.798" x2="22.987" y2="32.258" width="0.508" layer="1"/>
+<wire x1="9.57" y1="33.61" x2="9.57" y2="29.038" width="0.1524" layer="1"/>
+<wire x1="9.57" y1="29.038" x2="12.192" y2="26.416" width="0.1524" layer="1"/>
+<wire x1="12.192" y1="26.416" x2="14.732" y2="26.416" width="0.1524" layer="1"/>
+<wire x1="14.732" y1="26.416" x2="18.796" y2="30.48" width="0.1524" layer="1"/>
 </signal>
 <signal name="N$5">
@@
 <wire x1="3.49" y1="51.496" x2="4.064" y2="52.07" width="0.4572" layer="1"/>
 </signal>
-<signal name="BUCK_OUT" class="1">
-<contactref element="L_OUT" pad="P$2"/>
-<contactref element="C_OUT" pad="1"/>
-<contactref element="T2" pad="P$1"/>
-<contactref element="PWR" pad="A"/>
-<contactref element="DOUT" pad="A"/>
-<wire x1="18.796" y1="30.48" x2="18.796" y2="34.798" width="0.508" layer="1"/>
-<wire x1="18.796" y1="34.798" x2="18.796" y2="36.706" width="0.508" layer="1"/>
-<wire x1="18.796" y1="36.706" x2="18.92" y2="36.83" width="0.508" layer="1"/>
-<wire x1="18.92" y1="36.83" x2="18.92" y2="44.397" width="0.508" layer="1"/>
-<wire x1="18.92" y1="44.397" x2="18.973" y2="44.45" width="0.508" layer="1"/>
-<wire x1="18.973" y1="44.45" x2="22.86" y2="44.45" width="0.508" layer="1"/>
-<wire x1="22.86" y1="44.45" x2="22.987" y2="44.323" width="0.508" layer="1"/>
-<wire x1="18.796" y1="34.798" x2="20.447" y2="34.798" width="0.508" layer="1"/>
-<wire x1="20.447" y1="34.798" x2="22.987" y2="32.258" width="0.508" layer="1"/>
-</signal>
 </signals>
 <mfgpreviewcolors>
@@
 <mfgpreviewcolor name="substratecolor" color="0xFF786E46"/>
 </mfgpreviewcolors>
-<errors>
-</errors>
 </board>
 </drawing>
