File: PCBs/ElectroII (UPDATE).sch (EAGLE design)
At the start: 33 parts, among them IC1 TLF50211ELXUMA2, J1 U.FL-R-SMT(01), T1 VBAT, T2 BUCK, T3 GND, T5 VCC, T7 5V, U1 RFM95W-868S2

Commit message: fixed with erc and drc
should be go to go
Connections:
- removed net BUCK_OUT: C_OUT.1, DOUT.A, L_OUT.2, PWR.A, T2.P$1
- net FB: now also C_OUT.1, DOUT.A, L_OUT.2, PWR.A, T2.P$1
Changed lines of the file:
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@@
 <label x="81.28" y="-106.68" size="1.778" layer="95"/>
 <pinref part="IC1" gate="G$1" pin="FB"/>
+<pinref part="L_OUT" gate="G$1" pin="2"/>
+<wire x1="144.78" y1="-96.52" x2="147.32" y2="-96.52" width="0.1524" layer="91"/>
+<label x="152.4" y="-96.52" size="1.778" layer="95"/>
+<pinref part="C_OUT" gate="G$1" pin="1"/>
+<junction x="152.4" y="-96.52"/>
+<wire x1="147.32" y1="-96.52" x2="152.4" y2="-96.52" width="0.1524" layer="91"/>
+<wire x1="152.4" y1="-96.52" x2="172.72" y2="-96.52" width="0.1524" layer="91"/>
+<pinref part="T2" gate="G$1" pin="P$1"/>
+<pinref part="PWR" gate="G$1" pin="A"/>
+<wire x1="172.72" y1="-96.52" x2="177.8" y2="-96.52" width="0.1524" layer="91"/>
+<junction x="172.72" y="-96.52"/>
+<pinref part="DOUT" gate="1" pin="A"/>
+<wire x1="177.8" y1="-96.52" x2="193.04" y2="-96.52" width="0.1524" layer="91"/>
+<junction x="177.8" y="-96.52"/>
 <wire x1="71.12" y1="-109.22" x2="147.32" y2="-109.22" width="0.1524" layer="91"/>
 <wire x1="147.32" y1="-109.22" x2="147.32" y2="-96.52" width="0.1524" layer="91"/>
+<junction x="147.32" y="-96.52"/>
 </segment>
 </net>
@@
 </segment>
 </net>
-<net name="BUCK_OUT" class="1">
-<segment>
-<pinref part="L_OUT" gate="G$1" pin="2"/>
-<wire x1="144.78" y1="-96.52" x2="152.4" y2="-96.52" width="0.1524" layer="91"/>
-<label x="152.4" y="-96.52" size="1.778" layer="95"/>
-<pinref part="C_OUT" gate="G$1" pin="1"/>
-<junction x="152.4" y="-96.52"/>
-<wire x1="152.4" y1="-96.52" x2="172.72" y2="-96.52" width="0.1524" layer="91"/>
-<pinref part="T2" gate="G$1" pin="P$1"/>
-<pinref part="PWR" gate="G$1" pin="A"/>
-<wire x1="172.72" y1="-96.52" x2="177.8" y2="-96.52" width="0.1524" layer="91"/>
-<junction x="172.72" y="-96.52"/>
-<pinref part="DOUT" gate="1" pin="A"/>
-<wire x1="177.8" y1="-96.52" x2="193.04" y2="-96.52" width="0.1524" layer="91"/>
-<junction x="177.8" y="-96.52"/>
-</segment>
-</net>
