File: PCBs/Sensor Breakout Boards/Altimeter/Altimeter.brd (EAGLE design)
At the start: 25.4 x 25.4 mm, 2 parts, among them J1 2X6 FEMALE

Commit message: altimeter breakout v2
Parts:
- U$1: value ALTIMETER -> MS5803; device my-library:ALTIMETER -> MS5803:MS5803
- moved U$1 4.58 mm to (12.7, 8.89)
Connections:
- net N$1 renamed SDA
- net N$2 renamed SCL
- removed net N$3: J1.1, U$1.P$5
- removed net N$4: J1.11, U$1.P$2
- removed net N$5: J1.4, U$1.P$3
- removed net N$6: J1.6, U$1.P$6
- new net GND: J1.11, U$1.P$2, U$1.P$3
- new net VCC: J1.1, U$1.P$5, U$1.P$6
Routing:
- net N$6: track 63.7 -> 0.00 mm, vias 2 -> 0
- net N$5: track 48.9 -> 0.00 mm
- net VCC: track 0.00 -> 15.4 mm
- net GND: track 0.00 -> 12.7 mm
- net N$4: track 11.0 -> 0.00 mm
- net N$3: track 11.0 -> 0.00 mm, vias 2 -> 0
- net SCL: track 13.0 -> 10.4 mm
Changed lines of the file:
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@@
 <?xml version="1.0" encoding="utf-8"?>
 <!DOCTYPE eagle SYSTEM "eagle.dtd">
-<eagle version="9.5.1">
+<eagle version="9.5.0">
 <drawing>
 <settings>
@@
 <setting verticaltext="up"/>
 </settings>
-<grid distance="5" unitdist="mil" unit="mil" style="lines" multiple="1" display="no" altdistance="5" altunitdist="mil" altunit="inch"/>
+<grid distance="50" unitdist="mil" unit="mil" style="lines" multiple="1" display="no" altdistance="5" altunitdist="mil" altunit="inch"/>
 <layers>
 <layer number="1" name="Top" color="4" fill="1" visible="yes" active="yes"/>
@@
 <attribute name="VALUE" x="2.54" y="15.367" size="0.6096" layer="27" font="vector" ratio="20"/>
 </element>
-<element name="U$1" library="my-library" package="ALTIMETER" value="ALTIMETER" x="10.16" y="12.7" smashed="yes"/>
+<element name="U$1" library="MS5803" package="MS5803" value="MS5803" x="12.7" y="8.89" smashed="yes"/>
 </elements>
 <signals>
-<signal name="N$1">
+<signal name="SDA">
 <contactref element="J1" pad="3"/>
 <contactref element="U$1" pad="P$7"/>
-<wire x1="6.35" y1="17.78" x2="5.969" y2="17.399" width="0.508" layer="1"/>
-<wire x1="5.969" y1="17.399" x2="5.969" y2="11.811" width="0.508" layer="1"/>
-<wire x1="7.63" y1="10.15" x2="10.16" y2="10.15" width="0.508" layer="1"/>
-<wire x1="5.969" y1="11.811" x2="7.63" y2="10.15" width="0.508" layer="1"/>
+<wire x1="10.275" y1="9.54" x2="8.24" y2="9.54" width="0.4572" layer="1"/>
+<wire x1="8.24" y1="9.54" x2="6.35" y2="11.43" width="0.4572" layer="1"/>
+<wire x1="6.35" y1="11.43" x2="6.35" y2="17.78" width="0.4572" layer="1"/>
 </signal>
-<signal name="N$2">
+<signal name="VCC">
+<contactref element="J1" pad="1"/>
+<contactref element="U$1" pad="P$5"/>
+<contactref element="U$1" pad="P$6"/>
+<wire x1="10.275" y1="8.24" x2="7" y2="8.24" width="0.4572" layer="1"/>
+<wire x1="7" y1="8.24" x2="3.81" y2="11.43" width="0.4572" layer="1"/>
+<wire x1="3.81" y1="11.43" x2="3.81" y2="17.78" width="0.4572" layer="1"/>
+<wire x1="10.275" y1="6.99" x2="10.275" y2="8.24" width="0.4572" layer="1"/>
+</signal>
+<signal name="GND">
+<contactref element="J1" pad="11"/>
+<contactref element="U$1" pad="P$3"/>
+<contactref element="U$1" pad="P$2"/>
+<wire x1="14.85" y1="9.54" x2="15.125" y2="9.265" width="0.4572" layer="1"/>
+<wire x1="15.125" y1="9.265" x2="15.125" y2="8.24" width="0.4572" layer="1"/>
+<wire x1="14.85" y1="9.54" x2="17.16" y2="9.54" width="0.4572" layer="1"/>
+<wire x1="17.16" y1="9.54" x2="17.78" y2="10.16" width="0.4572" layer="1"/>
+<wire x1="17.78" y1="16.51" x2="16.51" y2="17.78" width="0.4572" layer="1"/>
+<wire x1="17.78" y1="10.16" x2="17.78" y2="16.51" width="0.4572" layer="1"/>
+</signal>
+<signal name="SCL">
 <contactref element="J1" pad="5"/>
 <contactref element="U$1" pad="P$1"/>
-<wire x1="8.89" y1="17.78" x2="12.0998" y2="14.5702" width="0.508" layer="1"/>
-<wire x1="12.0998" y1="14.5702" x2="12.0998" y2="9.906" width="0.508" layer="1"/>
-<wire x1="12.0998" y1="9.906" x2="13.1058" y2="8.9" width="0.508" layer="1"/>
-<wire x1="13.1058" y1="8.9" x2="15.46" y2="8.9" width="0.508" layer="1"/>
-</signal>
-<signal name="N$3">
-<contactref element="U$1" pad="P$5"/>
-<contactref element="J1" pad="1"/>
-<wire x1="10.16" y1="12.7" x2="8.89" y2="13.97" width="0.508" layer="1"/>
-<via x="8.89" y="13.97" extent="1-16" drill="0.79375"/>
-<wire x1="8.89" y1="13.97" x2="8.18438125" y2="13.97" width="0.4572" layer="16"/>
-<wire x1="8.18438125" y1="13.97" x2="7.40650625" y2="14.747875" width="0.4572" layer="16"/>
-<wire x1="7.40650625" y1="14.747875" x2="6.492875" y2="14.747875" width="0.508" layer="16"/>
-<wire x1="6.492875" y1="14.747875" x2="5.715" y2="13.97" width="0.508" layer="16"/>
-<wire x1="5.715" y1="13.97" x2="4.445" y2="13.97" width="0.508" layer="16"/>
-<wire x1="3.81" y1="17.78" x2="3.81" y2="14.605" width="0.508" layer="1"/>
-<wire x1="3.81" y1="14.605" x2="4.445" y2="13.97" width="0.508" layer="1"/>
-<via x="4.445" y="13.97" extent="1-16" drill="0.79375"/>
-</signal>
-<signal name="N$4">
-<contactref element="J1" pad="11"/>
-<contactref element="U$1" pad="P$2"/>
-<wire x1="16.51" y1="17.78" x2="16.51" y2="16.764" width="0.4572" layer="1"/>
-<wire x1="16.51" y1="16.764" x2="13.1412" y2="13.3952" width="0.508" layer="1"/>
-<wire x1="13.1412" y1="10.66993125" x2="13.66113125" y2="10.15" width="0.508" layer="1"/>
-<wire x1="13.66113125" y1="10.15" x2="15.46" y2="10.15" width="0.508" layer="1"/>
-<wire x1="13.1412" y1="10.66993125" x2="13.1412" y2="13.3952" width="0.508" layer="1"/>
-</signal>
-<signal name="N$5">
-<contactref element="U$1" pad="P$3"/>
-<contactref element="J1" pad="4"/>
-<wire x1="6.35" y1="20.32" x2="3.81" y2="22.86" width="0.508" layer="1"/>
-<wire x1="3.81" y1="22.86" x2="2.54" y2="22.86" width="0.508" layer="1"/>
-<wire x1="2.54" y1="22.86" x2="1.27" y2="21.59" width="0.508" layer="1"/>
-<wire x1="1.27" y1="21.59" x2="1.27" y2="7.62" width="0.508" layer="1"/>
-<wire x1="20.32" y1="7.62" x2="20.32" y2="10.16" width="0.508" layer="1"/>
-<wire x1="19.03" y1="11.45" x2="15.21" y2="11.45" width="0.508" layer="1"/>
-<wire x1="20.32" y1="10.16" x2="19.03" y2="11.45" width="0.508" layer="1"/>
-<wire x1="1.27" y1="7.62" x2="2.54" y2="6.35" width="0.508" layer="1"/>
-<wire x1="2.54" y1="6.35" x2="19.05" y2="6.35" width="0.508" layer="1"/>
-<wire x1="19.05" y1="6.35" x2="20.32" y2="7.62" width="0.508" layer="1"/>
-</signal>
-<signal name="N$6">
-<contactref element="U$1" pad="P$6"/>
-<contactref element="J1" pad="6"/>
-<wire x1="8.89" y1="20.32" x2="11.43" y2="22.86" width="0.508" layer="1"/>
-<wire x1="11.43" y1="22.86" x2="22.86" y2="22.86" width="0.508" layer="1"/>
-<wire x1="22.86" y1="22.86" x2="24.13" y2="21.59" width="0.508" layer="1"/>
-<wire x1="24.13" y1="21.59" x2="24.13" y2="5.08" width="0.508" layer="1"/>
-<wire x1="22.844125" y1="3.794125" x2="24.13" y2="5.08" width="0.508" layer="1"/>
-<via x="7.635875" y="12.7" extent="1-16" drill="0.79375"/>
-<wire x1="6.3579375" y1="11.4220625" x2="7.635875" y2="12.7" width="0.508" layer="16"/>
-<wire x1="7.635875" y1="12.7" x2="8.885875" y2="11.45" width="0.508" layer="1"/>
-<wire x1="8.885875" y1="11.45" x2="10.16" y2="11.45" width="0.4572" layer="1"/>
-<wire x1="6.492875" y1="4.429125" x2="6.477" y2="4.429125" width="0.4572" layer="1"/>
-<via x="6.477" y="4.429125" extent="1-16" drill="0.79375"/>
-<wire x1="6.3579375" y1="11.4220625" x2="6.477" y2="11.303" width="0.508" layer="16"/>
-<wire x1="6.477" y1="11.303" x2="6.477" y2="4.429125" width="0.508" layer="16"/>
-<wire x1="6.477" y1="4.429125" x2="7.096125" y2="3.81" width="0.508" layer="1"/>
-<wire x1="22.82825" y1="3.81" x2="22.844125" y2="3.794125" width="0.508" layer="1"/>
-<wire x1="7.096125" y1="3.81" x2="22.82825" y2="3.81" width="0.508" layer="1"/>
+<wire x1="15.125" y1="10.79" x2="13.63986875" y2="10.79" width="0.4572" layer="1"/>
+<wire x1="8.89" y1="15.53986875" x2="8.89" y2="17.78" width="0.4572" layer="1"/>
+<wire x1="13.63986875" y1="10.79" x2="8.89" y2="15.53986875" width="0.4572" layer="1"/>
 </signal>
 </signals>
