File: PCBs/Sensor Breakout Boards/Altimeter/Altimeter.sch (EAGLE design)
At the start: 2 parts, among them J1 2X6 FEMALE

Commit message: altimeter breakout v2
Parts:
- U$1: value ALTIMETER -> MS5803; device my-library:ALTIMETER -> MS5803:MS5803
Connections:
- net N$2 renamed SCL
- removed net N$1: J1.3, U$1.SDI/SDA
- removed net N$3: J1.1, U$1.VDD
- removed net N$4: J1.11, U$1.GND
- removed net N$5: J1.4, U$1.CSB
- removed net N$6: J1.6, U$1.PS
- new net GND: J1.11, U$1.CSB, U$1.GND
- new net SDA: J1.3, U$1.SDA/SDI
- new net VCC: J1.1, U$1.PS, U$1.VDD
Changed lines of the file:
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@@
 <parts>
 <part name="J1" library="RTR" deviceset="SENSOR_BREAKOUT" device="PTH_FEMALE" package3d_urn="urn:adsk.eagle:package:38277/1" value="2X6 FEMALE"/>
-<part name="U$1" library="my-library" deviceset="ALTIMETER" device=""/>
+<part name="GND2" library="RTR Main Library" deviceset="GND" device=""/>
+<part name="P+1" library="RTR Main Library" deviceset="VCC" device=""/>
+<part name="U$1" library="MS5803" deviceset="MS5803" device=""/>
+<part name="P+2" library="RTR Main Library" deviceset="VCC" device=""/>
+<part name="GND1" library="RTR Main Library" deviceset="GND" device=""/>
 </parts>
 <sheets>
@@
 <attribute name="NAME" x="59.69" y="81.788" size="1.778" layer="95" font="vector"/>
 </instance>
-<instance part="U$1" gate="G$1" x="66.04" y="5.08" smashed="yes">
-<attribute name="NAME" x="60.96" y="33.02" size="1.778" layer="95"/>
-<attribute name="VALUE" x="60.96" y="-25.4" size="1.778" layer="96"/>
+<instance part="GND2" gate="1" x="50.8" y="63.5" smashed="yes">
+<attribute name="VALUE" x="48.26" y="60.96" size="1.778" layer="96"/>
+</instance>
+<instance part="P+1" gate="VCC" x="55.88" y="81.28" smashed="yes">
+<attribute name="VALUE" x="53.34" y="78.74" size="1.778" layer="96" rot="R90"/>
+</instance>
+<instance part="U$1" gate="G$1" x="66.04" y="15.24" smashed="yes"/>
+<instance part="P+2" gate="VCC" x="43.18" y="27.94" smashed="yes">
+<attribute name="VALUE" x="40.64" y="25.4" size="1.778" layer="96" rot="R90"/>
+</instance>
+<instance part="GND1" gate="1" x="43.18" y="2.54" smashed="yes">
+<attribute name="VALUE" x="40.64" y="0" size="1.778" layer="96"/>
 </instance>
 </instances>
@@
 </busses>
 <nets>
-<net name="N$1" class="0">
+<net name="SDA" class="0">
 <segment>
 <pinref part="J1" gate="G$1" pin="3"/>
-<wire x1="55.88" y1="76.2" x2="30.48" y2="76.2" width="0.1524" layer="91"/>
-<wire x1="30.48" y1="76.2" x2="30.48" y2="0" width="0.1524" layer="91"/>
-<pinref part="U$1" gate="G$1" pin="SDI/SDA"/>
-<wire x1="30.48" y1="0" x2="40.64" y2="0" width="0.1524" layer="91"/>
+<wire x1="55.88" y1="76.2" x2="40.64" y2="76.2" width="0.1524" layer="91"/>
+<label x="40.64" y="76.2" size="1.778" layer="95"/>
+</segment>
+<segment>
+<pinref part="U$1" gate="G$1" pin="SDA/SDI"/>
+<wire x1="88.9" y1="17.78" x2="96.52" y2="17.78" width="0.1524" layer="91"/>
+<label x="96.52" y="17.78" size="1.778" layer="95"/>
 </segment>
 </net>
-<net name="N$2" class="0">
+<net name="VCC" class="0">
+<segment>
+<pinref part="J1" gate="G$1" pin="1"/>
+<pinref part="P+1" gate="VCC" pin="VCC"/>
+</segment>
+<segment>
+<pinref part="U$1" gate="G$1" pin="VDD"/>
+<pinref part="P+2" gate="VCC" pin="VCC"/>
+<pinref part="U$1" gate="G$1" pin="PS"/>
+<wire x1="43.18" y1="25.4" x2="43.18" y2="17.78" width="0.1524" layer="91"/>
+<junction x="43.18" y="25.4"/>
+</segment>
+</net>
+<net name="GND" class="0">
+<segment>
+<pinref part="J1" gate="G$1" pin="11"/>
+<pinref part="GND2" gate="1" pin="GND"/>
+<wire x1="55.88" y1="66.04" x2="50.8" y2="66.04" width="0.1524" layer="91"/>
+</segment>
+<segment>
+<pinref part="U$1" gate="G$1" pin="CSB"/>
+<pinref part="U$1" gate="G$1" pin="GND"/>
+<wire x1="43.18" y1="12.7" x2="43.18" y2="5.08" width="0.1524" layer="91"/>
+<pinref part="GND1" gate="1" pin="GND"/>
+<junction x="43.18" y="5.08"/>
+</segment>
+</net>
+<net name="SCL" class="0">
 <segment>
 <pinref part="J1" gate="G$1" pin="5"/>
 <wire x1="55.88" y1="73.66" x2="48.26" y2="73.66" width="0.1524" layer="91"/>
-<wire x1="48.26" y1="73.66" x2="48.26" y2="40.64" width="0.1524" layer="91"/>
-<wire x1="48.26" y1="40.64" x2="104.14" y2="40.64" width="0.1524" layer="91"/>
-<wire x1="104.14" y1="40.64" x2="104.14" y2="-10.16" width="0.1524" layer="91"/>
+<label x="48.26" y="73.66" size="1.778" layer="95"/>
+</segment>
+<segment>
 <pinref part="U$1" gate="G$1" pin="SCLK"/>
-<wire x1="104.14" y1="-10.16" x2="91.44" y2="-10.16" width="0.1524" layer="91"/>
+<wire x1="88.9" y1="22.86" x2="96.52" y2="22.86" width="0.1524" layer="91"/>
+<label x="96.52" y="22.86" size="1.778" layer="95"/>
 </segment>
 </net>
-<net name="N$3" class="0">
-<segment>
-<pinref part="U$1" gate="G$1" pin="VDD"/>
-<wire x1="40.64" y1="20.32" x2="22.86" y2="20.32" width="0.1524" layer="91"/>
-<pinref part="J1" gate="G$1" pin="1"/>
-<wire x1="22.86" y1="20.32" x2="22.86" y2="78.74" width="0.1524" layer="91"/>
-<wire x1="22.86" y1="78.74" x2="55.88" y2="78.74" width="0.1524" layer="91"/>
-</segment>
-</net>
-<net name="N$4" class="0">
-<segment>
-<pinref part="J1" gate="G$1" pin="11"/>
-<wire x1="55.88" y1="66.04" x2="40.64" y2="66.04" width="0.1524" layer="91"/>
-<wire x1="40.64" y1="66.04" x2="40.64" y2="93.98" width="0.1524" layer="91"/>
-<wire x1="40.64" y1="93.98" x2="111.76" y2="93.98" width="0.1524" layer="91"/>
-<wire x1="111.76" y1="93.98" x2="111.76" y2="0" width="0.1524" layer="91"/>
-<pinref part="U$1" gate="G$1" pin="GND"/>
-<wire x1="111.76" y1="0" x2="91.44" y2="0" width="0.1524" layer="91"/>
-</segment>
-</net>
-<net name="N$5" class="0">
-<segment>
-<pinref part="U$1" gate="G$1" pin="CSB"/>
-<wire x1="91.44" y1="10.16" x2="99.06" y2="10.16" width="0.1524" layer="91"/>
-<pinref part="J1" gate="G$1" pin="4"/>
-<wire x1="99.06" y1="10.16" x2="99.06" y2="76.2" width="0.1524" layer="91"/>
-<wire x1="99.06" y1="76.2" x2="71.12" y2="76.2" width="0.1524" layer="91"/>
-</segment>
-</net>
-<net name="N$6" class="0">
-<segment>
-<pinref part="U$1" gate="G$1" pin="PS"/>
-<wire x1="40.64" y1="10.16" x2="35.56" y2="10.16" width="0.1524" layer="91"/>
-<wire x1="35.56" y1="10.16" x2="35.56" y2="-35.56" width="0.1524" layer="91"/>
-<wire x1="35.56" y1="-35.56" x2="121.92" y2="-35.56" width="0.1524" layer="91"/>
-<pinref part="J1" gate="G$1" pin="6"/>
-<wire x1="121.92" y1="-35.56" x2="121.92" y2="73.66" width="0.1524" layer="91"/>
-<wire x1="121.92" y1="73.66" x2="71.12" y2="73.66" width="0.1524" layer="91"/>
-</segment>
-</net>
