File: PCBs/Sensor Breakout Boards/IMU_BNO055/BNO055_SCH.sch (EAGLE design)
At the start: 8 parts, among them U1 BNO055

Commit message: Updated Sketch
Parts:
- removed R2, R3: 10k, rcl:R-US_R1206
Connections:
- removed net ADDR_SEL: U1.COM3
- net BOOT: now also R1.1; no longer R2.2
- net GND: now also U1.COM3
- net SCL: no longer R1.2
- net SDA: no longer R3.2
- net VCC: now also R1.2; no longer R1.1, R2.1, R3.1
Other:
- moved on the sheet: R1
Changed lines of the file:
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@@
 <part name="C3" library="rcl" library_urn="urn:adsk.eagle:library:334" deviceset="C-US" device="C1206" package3d_urn="urn:adsk.eagle:package:23618/2" value="120 nF"/>
 <part name="GND4" library="supply1" library_urn="urn:adsk.eagle:library:371" deviceset="GND" device=""/>
-<part name="R1" library="rcl" library_urn="urn:adsk.eagle:library:334" deviceset="R-US_" device="R1206" package3d_urn="urn:adsk.eagle:package:23540/2" value="10k"/>
-<part name="R2" library="rcl" library_urn="urn:adsk.eagle:library:334" deviceset="R-US_" device="R1206" package3d_urn="urn:adsk.eagle:package:23540/2" value="10k"/>
-<part name="R3" library="rcl" library_urn="urn:adsk.eagle:library:334" deviceset="R-US_" device="R1206" package3d_urn="urn:adsk.eagle:package:23540/2" value="10k"/>
-<part name="P+3" library="supply1" library_urn="urn:adsk.eagle:library:371" deviceset="VCC" device=""/>
-<part name="P+4" library="supply1" library_urn="urn:adsk.eagle:library:371" deviceset="VCC" device=""/>
-<part name="P+5" library="supply1" library_urn="urn:adsk.eagle:library:371" deviceset="VCC" device=""/>
-<part name="GND5" library="supply1" library_urn="urn:adsk.eagle:library:371" deviceset="GND" device=""/>
 <part name="GND6" library="supply1" library_urn="urn:adsk.eagle:library:371" deviceset="GND" device=""/>
 <part name="GND7" library="supply1" library_urn="urn:adsk.eagle:library:371" deviceset="GND" device=""/>
@@
 <part name="P+6" library="supply1" library_urn="urn:adsk.eagle:library:371" deviceset="VCC" device=""/>
 <part name="GND8" library="supply1" library_urn="urn:adsk.eagle:library:371" deviceset="GND" device=""/>
+<part name="GND9" library="supply1" library_urn="urn:adsk.eagle:library:371" deviceset="GND" device=""/>
+<part name="R1" library="rcl" library_urn="urn:adsk.eagle:library:334" deviceset="R-US_" device="R1206" package3d_urn="urn:adsk.eagle:package:23540/2" value="10k"/>
+<part name="P+3" library="supply1" library_urn="urn:adsk.eagle:library:371" deviceset="VCC" device=""/>
 </parts>
 <sheets>
@@
 </instance>
 <instance part="GND1" gate="1" x="81.28" y="68.58" smashed="yes">
-<attribute name="VALUE" x="78.74" y="66.04" size="1.778" layer="96"/>
+<attribute name="VALUE" x="83.82" y="68.58" size="1.778" layer="96"/>
 </instance>
 <instance part="C1" gate="G$1" x="81.28" y="76.2" smashed="yes">
@@
 </instance>
 <instance part="GND3" gate="1" x="35.56" y="30.48" smashed="yes">
-<attribute name="VALUE" x="33.02" y="27.94" size="1.778" layer="96"/>
+<attribute name="VALUE" x="27.94" y="30.48" size="1.778" layer="96"/>
 </instance>
 <instance part="C3" gate="G$1" x="93.98" y="76.2" smashed="yes">
@@
 </instance>
 <instance part="GND4" gate="1" x="93.98" y="68.58" smashed="yes">
-<attribute name="VALUE" x="91.44" y="66.04" size="1.778" layer="96"/>
-</instance>
-<instance part="R1" gate="G$1" x="7.62" y="55.88" smashed="yes" rot="R270">
-<attribute name="NAME" x="9.1186" y="59.69" size="1.778" layer="95" rot="R270"/>
-<attribute name="VALUE" x="4.318" y="59.69" size="1.778" layer="96" rot="R270"/>
-</instance>
-<instance part="R2" gate="G$1" x="22.86" y="60.96" smashed="yes" rot="R270">
-<attribute name="NAME" x="24.3586" y="64.77" size="1.778" layer="95" rot="R270"/>
-<attribute name="VALUE" x="19.558" y="64.77" size="1.778" layer="96" rot="R270"/>
-</instance>
-<instance part="R3" gate="G$1" x="15.24" y="58.42" smashed="yes" rot="R270">
-<attribute name="NAME" x="16.7386" y="62.23" size="1.778" layer="95" rot="R270"/>
-<attribute name="VALUE" x="11.938" y="62.23" size="1.778" layer="96" rot="R270"/>
-</instance>
-<instance part="P+3" gate="VCC" x="15.24" y="66.04" smashed="yes">
-<attribute name="VALUE" x="12.7" y="63.5" size="1.778" layer="96" rot="R90"/>
-</instance>
-<instance part="P+4" gate="VCC" x="22.86" y="68.58" smashed="yes">
-<attribute name="VALUE" x="20.32" y="66.04" size="1.778" layer="96" rot="R90"/>
-</instance>
-<instance part="P+5" gate="VCC" x="7.62" y="63.5" smashed="yes">
-<attribute name="VALUE" x="5.08" y="60.96" size="1.778" layer="96" rot="R90"/>
-</instance>
-<instance part="GND5" gate="1" x="25.4" y="40.64" smashed="yes">
-<attribute name="VALUE" x="22.86" y="38.1" size="1.778" layer="96"/>
+<attribute name="VALUE" x="96.52" y="68.58" size="1.778" layer="96"/>
 </instance>
 <instance part="GND6" gate="1" x="30.48" y="63.5" smashed="yes">
-<attribute name="VALUE" x="27.94" y="60.96" size="1.778" layer="96"/>
+<attribute name="VALUE" x="22.86" y="63.5" size="1.778" layer="96"/>
 </instance>
 <instance part="GND7" gate="1" x="30.48" y="68.58" smashed="yes">
-<attribute name="VALUE" x="27.94" y="66.04" size="1.778" layer="96"/>
+<attribute name="VALUE" x="22.86" y="68.58" size="1.778" layer="96"/>
 </instance>
 <instance part="2X8" gate="G$1" x="-22.86" y="55.88" smashed="yes" rot="R180">
@@
 <instance part="GND8" gate="1" x="-35.56" y="45.72" smashed="yes">
 <attribute name="VALUE" x="-38.1" y="43.18" size="1.778" layer="96"/>
+</instance>
+<instance part="GND9" gate="1" x="30.48" y="40.64" smashed="yes">
+<attribute name="VALUE" x="22.86" y="40.64" size="1.778" layer="96"/>
+</instance>
+<instance part="R1" gate="G$1" x="20.32" y="60.96" smashed="yes" rot="R90">
+<attribute name="NAME" x="18.8214" y="57.15" size="1.778" layer="95" rot="R90"/>
+<attribute name="VALUE" x="23.622" y="57.15" size="1.778" layer="96" rot="R90"/>
+</instance>
+<instance part="P+3" gate="VCC" x="20.32" y="68.58" smashed="yes">
+<attribute name="VALUE" x="17.78" y="66.04" size="1.778" layer="96" rot="R90"/>
 </instance>
 </instances>
@@
 </segment>
 <segment>
-<pinref part="R3" gate="G$1" pin="1"/>
-<pinref part="P+3" gate="VCC" pin="VCC"/>
-</segment>
-<segment>
-<pinref part="R2" gate="G$1" pin="1"/>
-<pinref part="P+4" gate="VCC" pin="VCC"/>
-</segment>
-<segment>
-<pinref part="R1" gate="G$1" pin="1"/>
-<pinref part="P+5" gate="VCC" pin="VCC"/>
-</segment>
-<segment>
 <pinref part="2X8" gate="G$1" pin="1"/>
 <wire x1="-30.48" y1="63.5" x2="-33.02" y2="63.5" width="0.1524" layer="91"/>
 <wire x1="-33.02" y1="63.5" x2="-33.02" y2="66.04" width="0.1524" layer="91"/>
 <pinref part="P+6" gate="VCC" pin="VCC"/>
+</segment>
+<segment>
+<pinref part="R1" gate="G$1" pin="2"/>
+<pinref part="P+3" gate="VCC" pin="VCC"/>
 </segment>
 </net>
@@
 <segment>
 <pinref part="U1" gate="G$1" pin="COM2"/>
-<wire x1="35.56" y1="48.26" x2="25.4" y2="48.26" width="0.1524" layer="91"/>
-<wire x1="25.4" y1="48.26" x2="25.4" y2="43.18" width="0.1524" layer="91"/>
-<pinref part="GND5" gate="1" pin="GND"/>
+<wire x1="35.56" y1="48.26" x2="30.48" y2="48.26" width="0.1524" layer="91"/>
+<pinref part="U1" gate="G$1" pin="COM3"/>
+<wire x1="35.56" y1="45.72" x2="30.48" y2="45.72" width="0.1524" layer="91"/>
+<wire x1="30.48" y1="45.72" x2="30.48" y2="43.18" width="0.1524" layer="91"/>
+<pinref part="GND9" gate="1" pin="GND"/>
+<wire x1="30.48" y1="48.26" x2="30.48" y2="45.72" width="0.1524" layer="91"/>
+<junction x="30.48" y="45.72"/>
 </segment>
 <segment>
@@
 <net name="BOOT" class="0">
 <segment>
-<pinref part="R2" gate="G$1" pin="2"/>
 <pinref part="U1" gate="G$1" pin="NBOOT_LOAD_PIN"/>
-<wire x1="22.86" y1="55.88" x2="35.56" y2="55.88" width="0.1524" layer="91"/>
-<label x="22.86" y="43.18" size="1.778" layer="95" rot="R90"/>
-<wire x1="22.86" y1="55.88" x2="22.86" y2="43.18" width="0.1524" layer="91"/>
-<junction x="22.86" y="55.88"/>
+<label x="25.4" y="55.88" size="1.778" layer="95"/>
+<pinref part="R1" gate="G$1" pin="1"/>
+<wire x1="20.32" y1="55.88" x2="35.56" y2="55.88" width="0.1524" layer="91"/>
 </segment>
 </net>
 <net name="SDA" class="0">
-<segment>
-<pinref part="U1" gate="G$1" pin="COM0"/>
-<pinref part="R3" gate="G$1" pin="2"/>
-<wire x1="35.56" y1="53.34" x2="15.24" y2="53.34" width="0.1524" layer="91"/>
-<wire x1="15.24" y1="53.34" x2="15.24" y2="43.18" width="0.1524" layer="91"/>
-<junction x="15.24" y="53.34"/>
-<label x="15.24" y="43.18" size="1.778" layer="95" rot="R90"/>
-</segment>
 <segment>
 <pinref part="2X8" gate="G$1" pin="3"/>
@@
 <label x="-38.1" y="60.96" size="1.778" layer="95"/>
 </segment>
+<segment>
+<pinref part="U1" gate="G$1" pin="COM0"/>
+<wire x1="35.56" y1="53.34" x2="25.4" y2="53.34" width="0.1524" layer="91"/>
+<label x="25.4" y="53.34" size="1.778" layer="95"/>
+</segment>
 </net>
 <net name="SCL" class="0">
-<segment>
-<pinref part="U1" gate="G$1" pin="COM1"/>
-<pinref part="R1" gate="G$1" pin="2"/>
-<wire x1="35.56" y1="50.8" x2="7.62" y2="50.8" width="0.1524" layer="91"/>
-<wire x1="7.62" y1="50.8" x2="7.62" y2="43.18" width="0.1524" layer="91"/>
-<junction x="7.62" y="50.8"/>
-<label x="7.62" y="43.18" size="1.778" layer="95" rot="R90"/>
-</segment>
 <segment>
 <pinref part="2X8" gate="G$1" pin="5"/>
@@
 <label x="-38.1" y="58.42" size="1.778" layer="95"/>
 </segment>
-</net>
-<net name="ADDR_SEL" class="0">
-<segment>
-<pinref part="U1" gate="G$1" pin="COM3"/>
-<wire x1="35.56" y1="45.72" x2="30.48" y2="45.72" width="0.1524" layer="91"/>
-<wire x1="30.48" y1="45.72" x2="30.48" y2="35.56" width="0.1524" layer="91"/>
-<label x="30.48" y="35.56" size="1.778" layer="95" rot="R90"/>
+<segment>
+<pinref part="U1" gate="G$1" pin="COM1"/>
+<wire x1="35.56" y1="50.8" x2="25.4" y2="50.8" width="0.1524" layer="91"/>
+<label x="25.4" y="50.8" size="1.778" layer="95"/>
 </segment>
 </net>
@@
 <pinref part="U1" gate="G$1" pin="INT"/>
 <wire x1="76.2" y1="58.42" x2="83.82" y2="58.42" width="0.1524" layer="91"/>
-<label x="83.82" y="58.42" size="1.778" layer="95"/>
+<label x="81.28" y="58.42" size="1.778" layer="95"/>
 </segment>
 <segment>
@@
 <segment>
 <pinref part="U1" gate="G$1" pin="NRESET"/>
-<wire x1="35.56" y1="60.96" x2="27.94" y2="60.96" width="0.1524" layer="91"/>
-<wire x1="27.94" y1="60.96" x2="27.94" y2="76.2" width="0.1524" layer="91"/>
-<label x="27.94" y="76.2" size="1.778" layer="95" rot="R90"/>
-</segment>
-</net>
+<wire x1="35.56" y1="60.96" x2="25.4" y2="60.96" width="0.1524" layer="91"/>
+<label x="30.48" y="60.96" size="1.778" layer="95" rot="R180"/>
+</segment>
+</net>
