File: avio_flight_instruments_meeting_1.kicad_pcb (KiCad board)
At the start: 2 copper layers, 103.3 x 151.9 mm, 58 parts, among them J1 Conn_01x02_Male, J2 Conn_Coaxial, U1 MS5803-01BA_Miniature_Altimet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, U2 DS3231M, U3 RFM96W-433S2, U4 M20050-1, U5 BNO055

Commit message: update 11_17
Parts:
- removed BT2: S8411-45R, avio_flight_instruments_meeting_1:BAT_S8411-45R
- removed D2: Green, LED_THT:LED_D3.0mm
- removed R12, R15: 10k, Resistor_SMD:R_1206_3216Metric
- removed R13, R17: 0, Resistor_SMD:R_1206_3216Metric
- removed R14, R16: 220, Resistor_SMD:R_1206_3216Metric
- C12: value 0.1u -> 10u
- C13, C14: value 22p -> 0.1u
- C4: value 10u -> 22p
- C5: value 0.1u -> 2.2u
- C7: value 2.2u -> 22p
- J1: moved to F.Cu
- R1: value 0 -> 4.7k
- R2, R5: value 4.7k -> 0
- R4: value 0 -> 4.7K
- R7: value 220 -> 0
- R8: value 0 -> 220
- R9: value 0 -> 10k
- TP1: value 3.3V -> SCL1
- TP10: value TestPoint -> MISO
- TP11: value TestPoint -> SCL0
- TP12: value TestPoint -> SDA0
- TP2: value TestPoint -> SDA1
- TP3: value TestPoint -> 3.3V
- TP4: value TestPoint -> Fix
- TP5: value TestPoint -> HW
- TP6: value BOOTN -> RX
- TP7: value I2C_SDA0 -> TX
- TP8: value I2C_SCL0 -> BOOTN
- TP9: value TestPoint -> MOSI
- U3: value RFM96W-433S2 -> M20050-1; footprint RF_Module:HOPERF_RFM9XW_SMD -> avio_flight_instruments_meeting_1:XCVR_M20050-1
- U4: value M20050-1 -> BNO080; footprint avio_flight_instruments_meeting_1:XCVR_M20050-1 -> avio_flight_instruments_meeting_1:IC_BNO080
- U5: value BNO055 -> RFM96W-433S2; footprint avio_flight_instruments_meeting_1:BNO085 -> RF_Module:HOPERF_RFM9XW_SMD
- moved TP6 207.6 mm to (31.5, 150.4)
- moved TP7 207.0 mm to (31.5, 154.4)
- moved U5 185.9 mm to (50.0, 145.0), turned to 0 degrees
- moved C12 180.4 mm to (63.0, 144.5), turned to 180 degrees
- moved R6 152.5 mm to (26.2, 185.4), turned to 180 degrees
- moved C14 148.8 mm to (96.5, 150.6)
- moved C4 146.6 mm to (23.6, 180.6)
- moved U3 146.1 mm to (19.1, 166.4), turned to 90 degrees
- moved C5 146.1 mm to (29.2, 180.6)
- moved TP8 144.4 mm to (96.8, 138.7), turned to 0 degrees
- moved R5 143.8 mm to (68.5, 185.4)
- moved TP4 142.4 mm to (31.5, 162.1), turned to 90 degrees
- moved J2 135.7 mm to (26.4, 138.9), turned to 0 degrees
- moved TP5 135.6 mm to (31.5, 158.2), turned to 90 degrees
- moved U2 135.4 mm to (82.8, 183.1)
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Connections:
- A1 pad 12: RST-GPS -> FIX Indicator
- A1 pad 16: RST-TRX -> HW Standby
- A1 pad 18: DIO0 -> BOOTN
- A1 pad 22: unconnected-(A1-Pad22) -> INTN
- A1 pad 24: CS -> unconnected-(A1-Pad24)
- A1 pad 29: BOOTN -> CS
- A1 pad 31: INTN -> RST-TRX
- A1 pad 32: unconnected-(A1-Pad32) -> NRST
- A1 pad 33: NRST -> DIO0
- A1 pad 35: FIX Indicator -> unconnected-(A1-Pad35)
- A1 pad 36: unconnected-(A1-Pad36) -> CLKSEL0
- BT1 pad P: Net-(BT1-PadP) -> BAT
- C12 pad 2: Net-(C11-Pad2) -> Net-(C12-Pad2)
- C13 pad 1: RX -> GND
- C13 pad 2: GND -> Net-(C12-Pad2)
- C14 pad 1: TX -> GND
- C14 pad 2: GND -> Net-(C11-Pad2)
- C3 pad 1: Net-(BT1-PadP) -> BAT
- C6 pad 1: GND -> Net-(C6-Pad1)
- C7 pad 2: Net-(C6-Pad2) -> BAT
- C8 pad 1: Net-(C8-Pad1) -> RX
- C8 pad 2: Net-(C8-Pad2) -> GND
- C9 pad 1: GND -> TX
- C9 pad 2: Net-(BT2-PadP) -> GND
- R1 pad 2: Net-(C1-Pad2) -> SDA1
- R10 pad 1: GND -> +3.3V
- R10 pad 2: Net-(R10-Pad2) -> Net-(C12-Pad2)
- R11 pad 2: Net-(R11-Pad2) -> Net-(C11-Pad2)
- R2 pad 1: Net-(R2-Pad1) -> +3.3V
- R2 pad 2: SDA1alt -> Net-(C1-Pad2)
- R3 pad 1: Net-(R3-Pad1) -> +3.3V
- R3 pad 2: SDA1 -> SCL1
- R4 pad 2: Net-(R3-Pad1) -> Net-(C1-Pad2)
- R5 pad 1: Net-(R3-Pad1) -> +3.3V
- R5 pad 2: SCL1 -> Net-(C2-Pad2)
- R6 pad 2: Net-(C2-Pad2) -> Net-(C4-Pad2)
- R7 pad 1: Net-(A1-Pad40) -> GND
- R7 pad 2: Net-(D1-Pad2) -> Net-(R7-Pad2)
- R8 pad 1: +3.3V -> Net-(A1-Pad40)
- R8 pad 2: Net-(C4-Pad2) -> Net-(D1-Pad2)
- R9 pad 2: Net-(C6-Pad2) -> BOOTN
- TP1 pad 1: +3.3V -> SCL1
- TP10 pad 1: FIX Indicator -> MISO0
- TP11 pad 1: RX -> SCL0
- TP12 pad 1: TX -> SDA0
- TP2 pad 1: SCL1 -> SDA1
- TP3 pad 1: SDA1 -> +3.3V
- TP4 pad 1: MOSI0 -> FIX Indicator
- TP5 pad 1: MISO0 -> HW Standby
- TP6 pad 1: BOOTN -> RX
- TP7 pad 1: SDA0 -> TX
- TP8 pad 1: SCL0 -> BOOTN
- TP9 pad 1: HW Standby -> MOSI0
- U1 pad 3: Net-(R2-Pad2) -> Net-(C1-Pad2)
- U1 pad 6: Net-(R2-Pad2) -> Net-(C1-Pad2)
- U2 pad 14: Net-(BT1-PadP) -> BAT
- U3 pad 1: GND -> Net-(R7-Pad2)
- U3 pad 10: GND -> unconnected-(U3-Pad10)
- U3 pad 12: unconnected-(U3-Pad12) -> BAT
- U3 pad 13: Net-(C4-Pad2) -> unconnected-(U3-Pad13)
- U3 pad 14: DIO0 -> unconnected-(U3-Pad14)
- U3 pad 15: unconnected-(U3-Pad15) -> GND
- U3 pad 16: unconnected-(U3-Pad16) -> GND
- U3 pad 2: MISO0 -> GND
- U3 pad 3: MOSI0 -> GND
- U3 pad 4: SCLK -> Net-(C6-Pad2)
- U3 pad 5: CS -> GND
- U3 pad 6: RST-TRX -> Net-(C6-Pad1)
- U3 pad 7: unconnected-(U3-Pad7) -> GND
- U3 pad 8: GND -> Net-(C4-Pad2)
- U3 pad 9: Net-(J2-Pad1) -> GND
- U4 pad 1: Net-(R10-Pad2) -> unconnected-(U4-Pad1)
- U4 pad 10: RST-GPS -> CLKSEL0
- U4 pad 11: unconnected-(U4-Pad11) -> NRST
- U4 pad 12: Net-(BT2-PadP) -> unconnected-(U4-Pad12)
- U4 pad 14: unconnected-(U4-Pad14) -> INTN
- U4 pad 15: GND -> unconnected-(U4-Pad15)
- U4 pad 16: GND -> unconnected-(U4-Pad16)
- U4 pad 18: FIX Indicator -> unconnected-(U4-Pad18)
- U4 pad 19: GND -> SCL0
- U4 pad 20: Net-(L3-Pad1) -> SDA0
- U4 pad 21: Net-(L2-Pad1) -> unconnected-(U4-Pad21)
- U4 pad 22: GND -> unconnected-(U4-Pad22)
- U4 pad 23: GND -> unconnected-(U4-Pad23)
- U4 pad 24: GND -> unconnected-(U4-Pad24)
- U4 pad 26: HW Standby -> unconnected-(U4-Pad26)
- U4 pad 27: GND -> unconnected-(U4-Pad27)
- U4 pad 28: Net-(L1-Pad2) -> Net-(C11-Pad2)
- U4 pad 3: GND -> Net-(C11-Pad2)
- U4 pad 4: Net-(C8-Pad2) -> BOOTN
- U4 pad 6: Net-(C8-Pad1) -> GND
- U4 pad 7: GND -> unconnected-(U4-Pad7)
- U4 pad 8: Net-(C6-Pad2) -> unconnected-(U4-Pad8)
- U4 pad 9: GND -> Net-(C10-Pad2)
- U5 pad 1: (no net) -> GND
- U5 pad 10: unconnected-(U5-Pad10) -> GND
- U5 pad 11: NRST -> unconnected-(U5-Pad11)
- U5 pad 12: (no net) -> unconnected-(U5-Pad12)
- U5 pad 13: (no net) -> Net-(C12-Pad2)
- U5 pad 14: INTN -> DIO0
- U5 pad 2: GND -> MISO0
- U5 pad 3: Net-(C11-Pad2) -> MOSI0
- U5 pad 4: BOOTN -> SCLK
- U5 pad 5: GND -> CS
- U5 pad 6: GND -> RST-TRX
- U5 pad 7: (no net) -> unconnected-(U5-Pad7)
- U5 pad 8: (no net) -> GND
- U5 pad 9: Net-(C10-Pad2) -> Net-(J2-Pad1)
Routing:
- added copper zone on B.Cu, net (none)
- added copper zone on F.Cu, net (none)
- added copper zone on In1.Cu, net (none)
- added copper zone on In2.Cu, net +3.3V
- removed copper zone on B.Cu, net GND
- removed copper zone on F.Cu, net GND
Other:
- board size 103.3 x 151.9 mm -> 102.2 x 63.6 mm
- copper layers 2 -> 4

Commit message: Added layout version 1 11_23_22
Parts:
- added A1: ADA3708, avio_flight_instruments_meeting_1:ADA3708_RPI-ZERO, F.Cu at (170.4, 106.1)
- added REF**: MountingHole_2.5mm, MountingHole:MountingHole_2.5mm, F.Cu at (105.4, 74.0)
- added REF**: MountingHole_2.5mm, MountingHole:MountingHole_2.5mm, F.Cu at (105.4, 129.2)
- added REF**: MountingHole_2.5mm, MountingHole:MountingHole_2.5mm, F.Cu at (199.4, 74.0)
- added REF**: MountingHole_3.5mm, MountingHole:MountingHole_3.5mm, B.Cu at (165.9, 96.5)
- added REF**: MountingHole_3.5mm, MountingHole:MountingHole_3.5mm, B.Cu at (139.2, 96.5)
- C1: value 100 nF -> 22p
- C11, C13: value 0.1u -> 0.47u
- C12: value 10u -> 0.1u
- C2: value 0.47u -> 2.2u
- C3: value 0.47u -> 22p
- C5: value 2.2u -> 10u
- C6: value 22p -> 0.1u
- C9: value 22p -> 100 nF
- J1: moved to B.Cu
- R1, R3: value 4.7k -> 0
- R4: value 4.7K -> 0
- R5: value 0 -> 4.7K
- R6: value 0 -> 220
- R7: value 0 -> 10k
- R8: value 220 -> 4.7k
- R9: value 10k -> 4.7k
- TP1: value SCL1 -> MOSI
- TP10: value MISO -> BOOTN
- TP2: value SDA1 -> MISO
- TP3: value 3.3V -> Fix
- TP4: value Fix -> HW
- TP5: value HW -> RX
- TP6: value RX -> TX
- TP7: value TX -> 3.3V
- TP8: value BOOTN -> SCL1
- TP9: value MOSI -> SDA1
- U1: value MS5803-01BA_Miniature_Altimeter_Module -> M20050-1; footprint avio_flight_instruments_meeting_1:MS5803-01BA_Miniature_Altimeter_Module -> avio_flight_instruments_meeting_1:XCVR_M20050-1
- U2: value DS3231M -> RFM96W-433S2; footprint avio_flight_instruments_meeting_1:SOIC127P1032X265-16N -> RF_Module:HOPERF_RFM9XW_SMD
- U3: value M20050-1 -> MS5803-01BA_Miniature_Altimeter_Module; footprint avio_flight_instruments_meeting_1:XCVR_M20050-1 -> avio_flight_instruments_meeting_1:MS5803-01BA_Miniature_Altimeter_Module
- U5: value RFM96W-433S2 -> DS3231M; footprint RF_Module:HOPERF_RFM9XW_SMD -> avio_flight_instruments_meeting_1:SOIC127P1032X265-16N
- moved R7 196.2 mm to (184.2, 78.5), turned to 0 degrees
- moved R6 189.1 mm to (194.6, 99.4), turned to 90 degrees
- moved C6 169.7 mm to (156.7, 83.8), turned to 0 degrees
- moved C5 157.4 mm to (151.1, 81.1), turned to 90 degrees
- moved BT1 156.8 mm to (191.9, 117.6), turned to 90 degrees
- moved TP10 152.5 mm to (179.7, 84.1)
- moved C12 145.0 mm to (189.2, 73.2)
- moved R3 126.5 mm to (156.7, 78.0), turned to 180 degrees
- moved C7 123.7 mm to (109.1, 84.3), turned to 90 degrees
- moved U5 123.6 mm to (170.9, 119.1)
- moved C4 122.0 mm to (120.1, 105.9), turned to 90 degrees
- moved C13 121.3 mm to (181.4, 123.7), turned to -90 degrees
- moved R11 118.6 mm to (184.2, 73.2), turned to 0 degrees
- moved C14 117.5 mm to (189.2, 78.5)
- moved C8 117.4 mm to (113.3, 84.3), turned to 90 degrees
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Connections:
- A1 pad 11: RST-RTC -> FIX
- A1 pad 12: FIX Indicator -> RST-TRX
- A1 pad 13: unconnected-(A1-Pad13) -> HW
- A1 pad 16: HW Standby -> CS
- A1 pad 18: BOOTN -> DIO0
- A1 pad 22: INTN -> BOOTN
- A1 pad 29: CS -> unconnected-(A1-Pad29)
- A1 pad 31: RST-TRX -> unconnected-(A1-Pad31)
- A1 pad 32: NRST -> CLKSEL0
- A1 pad 33: DIO0 -> unconnected-(A1-Pad33)
- A1 pad 36: CLKSEL0 -> NRST
- A1 pad 38: unconnected-(A1-Pad38) -> INTN
- A1 pad 7: unconnected-(A1-Pad7) -> RST-RTC
- C13 pad 1: GND -> BAT
- C13 pad 2: Net-(C12-Pad2) -> GND
- C14 pad 2: Net-(C11-Pad2) -> Net-(C12-Pad2)
- C2 pad 2: Net-(C2-Pad2) -> Net-(C1-Pad2)
- C3 pad 1: BAT -> Net-(C3-Pad1)
- C3 pad 2: GND -> Net-(C3-Pad2)
- C4 pad 2: Net-(C4-Pad2) -> BAT
- C5 pad 2: Net-(C4-Pad2) -> Net-(C5-Pad2)
- C6 pad 1: Net-(C6-Pad1) -> GND
- C6 pad 2: Net-(C6-Pad2) -> Net-(C5-Pad2)
- C7 pad 1: GND -> RX
- C7 pad 2: BAT -> GND
- C8 pad 1: RX -> TX
- C9 pad 1: TX -> GND
- C9 pad 2: GND -> Net-(C9-Pad2)
- R1 pad 2: SDA1 -> Net-(C1-Pad2)
- R10 pad 2: Net-(C12-Pad2) -> Net-(C11-Pad2)
- R11 pad 2: Net-(C11-Pad2) -> Net-(C12-Pad2)
- R2 pad 1: +3.3V -> GND
- R2 pad 2: Net-(C1-Pad2) -> Net-(R2-Pad2)
- R3 pad 2: SCL1 -> Net-(C5-Pad2)
- R4 pad 2: Net-(C1-Pad2) -> Net-(C9-Pad2)
- R5 pad 2: Net-(C2-Pad2) -> Net-(C9-Pad2)
- R6 pad 1: +3.3V -> Net-(A1-Pad40)
- R6 pad 2: Net-(C4-Pad2) -> Net-(D1-Pad2)
- R7 pad 1: GND -> +3.3V
- R7 pad 2: Net-(R7-Pad2) -> BOOTN
- R8 pad 1: Net-(A1-Pad40) -> +3.3V
- R8 pad 2: Net-(D1-Pad2) -> SDA1
- R9 pad 2: BOOTN -> SCL1
- TP1 pad 1: SCL1 -> MOSI0
- TP10 pad 1: MISO0 -> BOOTN
- TP2 pad 1: SDA1 -> MISO0
- TP3 pad 1: +3.3V -> FIX
- TP4 pad 1: FIX Indicator -> HW
- TP5 pad 1: HW Standby -> RX
- TP6 pad 1: RX -> TX
- TP7 pad 1: TX -> +3.3V
- TP8 pad 1: BOOTN -> SCL1
- TP9 pad 1: MOSI0 -> SDA1
- U1 pad 1: SCL1 -> Net-(R2-Pad2)
- U1 pad 3: Net-(C1-Pad2) -> GND
- U1 pad 4: unconnected-(U1-Pad4) -> Net-(C3-Pad2)
- U1 pad 5: Net-(C1-Pad2) -> GND
- U1 pad 6: Net-(C1-Pad2) -> Net-(C3-Pad1)
- U1 pad 7: SDA1 -> GND
- U1 pad 8: unconnected-(U1-Pad8) -> Net-(C1-Pad2)
- U2 pad 1: unconnected-(U2-Pad1) -> GND
- U2 pad 11: GND -> unconnected-(U2-Pad11)
- U2 pad 12: GND -> unconnected-(U2-Pad12)
- U2 pad 13: GND -> Net-(C5-Pad2)
- U2 pad 14: BAT -> DIO0
- U2 pad 15: SDA1 -> unconnected-(U2-Pad15)
- U2 pad 16: SCL1 -> unconnected-(U2-Pad16)
- U2 pad 2: Net-(C2-Pad2) -> MISO0
- U2 pad 3: unconnected-(U2-Pad3) -> MOSI0
- U2 pad 4: RST-RTC -> SCLK
- U2 pad 5: GND -> CS
- U2 pad 6: GND -> RST-TRX
- U2 pad 7: GND -> unconnected-(U2-Pad7)
- U2 pad 9: GND -> Net-(J2-Pad1)
- U3 pad 1: Net-(R7-Pad2) -> SCL1
- U3 pad 3: GND -> Net-(C9-Pad2)
- U3 pad 4: Net-(C6-Pad2) -> unconnected-(U3-Pad4)
- U3 pad 5: GND -> Net-(C9-Pad2)
- U3 pad 6: Net-(C6-Pad1) -> Net-(C9-Pad2)
- U3 pad 7: GND -> SDA1
- U3 pad 8: Net-(C4-Pad2) -> unconnected-(U3-Pad8)
- U4 pad 28: Net-(C11-Pad2) -> Net-(C12-Pad2)
- U4 pad 3: Net-(C11-Pad2) -> Net-(C12-Pad2)
- U5 pad 1: GND -> unconnected-(U5-Pad1)
- U5 pad 11: unconnected-(U5-Pad11) -> GND
- U5 pad 12: unconnected-(U5-Pad12) -> GND
- U5 pad 13: Net-(C12-Pad2) -> GND
- U5 pad 14: DIO0 -> BAT
- U5 pad 15: unconnected-(U5-Pad15) -> SDA1
- U5 pad 16: unconnected-(U5-Pad16) -> SCL1
- U5 pad 2: MISO0 -> Net-(C11-Pad2)
- U5 pad 3: MOSI0 -> unconnected-(U5-Pad3)
- U5 pad 4: SCLK -> RST-RTC
- U5 pad 5: CS -> GND
- U5 pad 6: RST-TRX -> GND
- U5 pad 7: unconnected-(U5-Pad7) -> GND
- U5 pad 9: Net-(J2-Pad1) -> GND
Routing:
- net HW: track 0.00 -> 155.0 mm, vias 0 -> 2
- net SDA1: track 0.00 -> 105.3 mm, vias 0 -> 2
- net MISO0: track 0.00 -> 105.0 mm, vias 0 -> 1
- net SCL1: track 0.00 -> 82.5 mm, vias 0 -> 2
- net BAT: track 0.00 -> 79.4 mm, vias 0 -> 1
- net MOSI0: track 0.00 -> 60.9 mm, vias 0 -> 1
- net RX: track 0.00 -> 60.8 mm, vias 0 -> 4
- net SCLK: track 0.00 -> 56.7 mm, vias 0 -> 1
- net CS: track 0.00 -> 55.0 mm, vias 0 -> 1
- net FIX: track 0.00 -> 54.2 mm, vias 0 -> 1
- net TX: track 0.00 -> 54.1 mm, vias 0 -> 3
- net SDA0: track 0.00 -> 52.1 mm, vias 0 -> 1
- net RST-TRX: track 0.00 -> 46.1 mm, vias 0 -> 1
- net BOOTN: track 0.00 -> 40.4 mm, vias 0 -> 1
- net SCL0: track 0.00 -> 39.2 mm, vias 0 -> 1
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- added copper zone on B.Cu, net GND
- added copper zone on F.Cu, net GND
- added copper zone on In1.Cu, net GND
- removed copper zone on B.Cu, net (none)
- removed copper zone on F.Cu, net (none)
- removed copper zone on In1.Cu, net (none)

Commit message: Neutro layout revision 12.2.22
Parts:
- removed the A1 at (170.4, 106.1) (x2)
- added A1: ADA3708, avio_flight_instruments_meeting_1:ADA3708_RPI-ZERO, B.Cu at (158.8, 90.4)
- added D2: Green, LED_THT:LED_D3.0mm, F.Cu at (135.0, 127.9)
- added R12: 0, Resistor_SMD:R_1206_3216Metric, F.Cu at (165.3, 74.8)
- added REF**: MountingHole_2.5mm, MountingHole:MountingHole_2.5mm, F.Cu at (199.4, 129.2)
- C5: value 10u -> locked
- D1: value Green -> Red
- R10: value 0 -> 4.7k
- R7: value 10k -> 220
- R8: value 4.7k -> 10k
- moved J2 90.9 mm to (198.1, 113.4), turned to -90 degrees
- moved R7 79.5 mm to (122.8, 129.0), turned to -90 degrees
- moved R6 72.8 mm to (126.0, 123.7), turned to -90 degrees
- moved BT1 72.1 mm to (121.5, 101.9), turned to -90 degrees
- moved D1 71.3 mm to (135.0, 122.4), turned to -90 degrees
- moved R11 60.4 mm to (135.3, 108.6), turned to -90 degrees
- moved TP2 56.0 mm to (158.9, 121.2)
- moved U2 55.2 mm to (174.8, 122.3)
- moved TP1 55.0 mm to (159.0, 128.4)
- moved R5 50.3 mm to (136.9, 77.3)
- moved C9 47.6 mm to (156.6, 80.3)
- moved U3 46.7 mm to (148.1, 80.4)
- moved R8 42.6 mm to (165.4, 79.1), turned to 0 degrees
- moved R4 41.1 mm to (137.1, 82.3)
- moved R3 40.6 mm to (182.9, 109.0), turned to -90 degrees
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Connections:
- R10 pad 2: Net-(C11-Pad2) -> SCL1
- R11 pad 2: Net-(C12-Pad2) -> Net-(C11-Pad2)
- R5 pad 1: +3.3V -> Net-(C9-Pad2)
- R7 pad 1: +3.3V -> Net-(A1-Pad40)
- R7 pad 2: BOOTN -> Net-(D2-Pad2)
- R8 pad 2: SDA1 -> BOOTN
- R9 pad 2: SCL1 -> SDA1
Routing:
- net HW: track 155.0 -> 39.3 mm, vias 2 -> 3
- net MISO0: track 105.0 -> 39.2 mm, vias 1 -> 2
- net SDA1: track 105.3 -> 43.0 mm, vias 2 -> 6
- net SCL1: track 82.5 -> 34.1 mm, vias 2 -> 5
- net Net-(A1-Pad40): track 0.00 -> 43.4 mm, vias 0 -> 1
- net Net-(A1-Pad38): track 3.87 -> 37.8 mm
- net BAT: track 79.4 -> 48.1 mm, vias 1 -> 7
- net +3.3V: track 0.00 -> 26.7 mm
- net SDA0: track 52.1 -> 26.8 mm, vias 1 -> 2
- net FIX: track 54.2 -> 29.8 mm, vias 1 -> 3
- net CS: track 55.0 -> 35.7 mm, vias 1 -> 3
- net MOSI0: track 60.9 -> 43.2 mm, vias 1 -> 3
- net SCLK: track 56.7 -> 40.1 mm, vias 1 -> 2
- net Net-(J2-Pad1): track 38.6 -> 23.7 mm
- net TX: track 54.1 -> 68.8 mm, vias 3 -> 5
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Other:
- board size 102.2 x 63.6 mm -> 101.6 x 63.5 mm
