File: avio_flight_instruments_meeting_1.kicad_pcb (KiCad board)
At the start: 4 copper layers, 101.6 x 63.5 mm, 58 parts, among them J1 Conn_01x02_Male, J2 Conn_Coaxial, U1 M20050-1, U2 RFM96W-433S2, U3 MS5803-01BA_Miniature_Altimet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, U4 BNO080, U5 DS3231M

Commit message: layout revision 12.4.22
Parts:
- C9: value 100 nF -> 100nF
- TP3: value Fix -> FIX
- moved C10 5.15 mm to (194.3, 81.4), turned to -90 degrees
- moved TP1 4.49 mm to (162.2, 125.2)
- moved TP2 4.34 mm to (157.4, 125.2)
- moved R8 3.23 mm to (164.3, 82.2)
- moved R12 3.23 mm to (164.2, 77.9)
- moved TP10 3.23 mm to (174.4, 82.0)
- moved TP11 3.23 mm to (189.4, 82.3)
- moved U4 3.23 mm to (182.1, 82.3)
- moved C12 3.23 mm to (181.6, 76.5)
- moved C14 3.23 mm to (174.4, 76.5)
- moved TP12 3.23 mm to (189.4, 76.5)
- moved C9 2.05 mm to (154.6, 80.3)
- moved R4 2.05 mm to (135.0, 82.3)
- moved R5 2.05 mm to (134.9, 77.3)
- moved U3 2.05 mm to (146.1, 80.4)
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Routing:
- net GND: track 0.00 -> 6.53 mm, vias 28 -> 33
- net Net-(C10-Pad2): track 9.36 -> 15.7 mm
- net +3.3V: track 26.7 -> 20.6 mm, vias 10 -> 8
- net SCL0: track 24.9 -> 20.0 mm
- net MISO0: track 39.2 -> 43.8 mm, vias 2 -> 3
- net MOSI0: track 43.2 -> 38.7 mm
- net BOOTN: track 30.9 -> 26.8 mm
- net INTN: track 18.8 -> 16.5 mm
- net NRST: track 22.4 -> 20.1 mm
- net CLKSEL0: track 25.0 -> 22.9 mm
- net SDA0: track 26.8 -> 25.0 mm
- net SCL1: track 34.1 -> 32.6 mm
- net BAT: track 48.1 -> 46.9 mm
- net Net-(C5-Pad2): track 22.4 -> 21.3 mm
- net SDA1: track 43.0 -> 42.1 mm
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
Commit message: Revision 12.24.22
Parts:
- removed REF** (x4): MountingHole_2.5mm, MountingHole:MountingHole_2.5mm
- removed REF** (x2): MountingHole_3.5mm, MountingHole:MountingHole_3.5mm
- added H1: MountingHole, MountingHole:MountingHole_2.5mm, F.Cu at (106.1, 74.5)
- added H2: MountingHole, MountingHole:MountingHole_2.5mm, F.Cu at (198.7, 74.4)
- added H3: MountingHole, MountingHole:MountingHole_2.5mm, F.Cu at (198.7, 129.0)
- added H4: MountingHole, MountingHole:MountingHole_2.5mm, F.Cu at (106.1, 129.0)
- added H5: MountingHole, MountingHole:MountingHole_3.5mm, F.Cu at (139.1, 100.1)
- added H6: MountingHole, MountingHole:MountingHole_3.5mm, F.Cu at (165.7, 100.1)
- C9: value 100nF -> 100 nF
- TP3: value FIX -> Fix
- moved J2 6.86 mm to (198.1, 120.3)
- moved D1 6.09 mm to (129.5, 119.8)
- moved D2 5.95 mm to (129.5, 125.6)
- moved R6 5.37 mm to (123.7, 118.8)
- moved L1 4.50 mm to (103.3, 93.1)
- moved R2 3.19 mm to (103.1, 109.8)
- moved R7 2.50 mm to (123.7, 126.7)
- moved C12 1.56 mm to (180.3, 75.5), turned to -90 degrees
- moved R4 1.02 mm to (134.0, 82.2)
- moved R5 0.88 mm to (134.0, 77.5)
Connections:
- R5 pad 2: Net-(C9-Pad2) -> Net-(R5-Pad2)
- U3 pad 3: Net-(C9-Pad2) -> Net-(R5-Pad2)
- U3 pad 6: Net-(C9-Pad2) -> Net-(R5-Pad2)
Routing:
- net GND: track 6.53 -> 38.4 mm, vias 33 -> 14
- net Net-(R5-Pad2): track 0.00 -> 13.8 mm, vias 0 -> 2
- net Net-(D2-Pad2): track 12.2 -> 5.83 mm
- net Net-(J2-Pad1): track 23.7 -> 19.1 mm
- net Net-(L1-Pad2): track 7.00 -> 2.99 mm, vias 2 -> 0
- net Net-(C9-Pad2): track 28.4 -> 32.1 mm
- net Net-(A1-Pad38): track 37.8 -> 34.7 mm
- net Net-(A1-Pad40): track 43.4 -> 40.7 mm
- net Net-(R2-Pad2): track 5.73 -> 3.18 mm, vias 2 -> 0
- net Net-(D1-Pad2): track 9.15 -> 6.66 mm
- net Net-(C12-Pad2): track 23.1 -> 24.0 mm, vias 6 -> 5
- net BAT: track 46.9 -> 47.8 mm
- net HW: track 39.2 -> 38.4 mm
Other:
- board text added: "Neutro"
- board text added: "Rice Eclipse"
- board text added: "v1"
