File: Neutro_v1.kicad_sch (KiCad schematic)
At the start: 61 parts, among them J1 SparkFun_Lipo_Converter, J2 Conn_Coaxial, U1 M20050-1, U2 RFM96W-433S2_1, U3 MS5803-01BA, U4 BNO080, U5 DS3231M_1

Commit message: neutro pcb v1 final design 1.21.22
Connections:
- net t_pwr: now reaches C5.2, C6.2, R3.2, U2.13 (3.3V)
- net gps_pwr: now reaches C1.2, C2.2, R1.2, U1.8 (VCC)
Changed lines of the file:
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@@
     (effects (font (size 2.5 2.5)) (justify left bottom))
+  )
+  (label "t_pwr" (at 81.28 93.98 0)
+    (effects (font (size 1.27 1.27)) (justify left bottom))
+  )
+  (label "gps_pwr" (at 41.91 201.93 0)
+    (effects (font (size 1.27 1.27)) (justify left bottom))
   )
   (global_label "INTN" (shape output) (at 370.84 96.52 0) (fields_autoplaced)

Commit message: neutro v1 1.21.23 final pcb (change L2, L3 size)
Parts:
- L2, L3: footprint Inductor_SMD:L_1206_3216Metric -> Inductor_SMD:L_1008_2520Metric
Changed lines of the file:
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@@
     (property "Reference" "L3" (id 0) (at 119.38 208.28 90))
     (property "Value" "47n" (id 1) (at 119.38 205.74 90))
-    (property "Footprint" "Inductor_SMD:L_1206_3216Metric" (id 2) (at 119.38 204.47 0)
+    (property "Footprint" "Inductor_SMD:L_1008_2520Metric" (id 2) (at 119.38 204.47 0)
       (effects (font (size 1.27 1.27)) hide)
     )
@@
     (property "Reference" "L2" (id 0) (at 106.68 196.85 90))
     (property "Value" "47n" (id 1) (at 106.68 199.39 90))
-    (property "Footprint" "Inductor_SMD:L_1206_3216Metric" (id 2) (at 106.68 201.93 0)
+    (property "Footprint" "Inductor_SMD:L_1008_2520Metric" (id 2) (at 106.68 201.93 0)
       (effects (font (size 1.27 1.27)) hide)
     )
@@
     )
     (path "/579f6778-0fa4-48c0-ace3-32fe62e6e30f"
-      (reference "L2") (unit 1) (value "47n") (footprint "Inductor_SMD:L_1206_3216Metric")
+      (reference "L2") (unit 1) (value "47n") (footprint "Inductor_SMD:L_1008_2520Metric")
     )
     (path "/3fbd9f02-b5c4-4403-8729-94c5f05e253a"
-      (reference "L3") (unit 1) (value "47n") (footprint "Inductor_SMD:L_1206_3216Metric")
+      (reference "L3") (unit 1) (value "47n") (footprint "Inductor_SMD:L_1008_2520Metric")
     )
     (path "/4d75ebbc-b2e2-4e56-bc2e-dc62c7c80fd4"
